File: 8bit_computer.sch (EAGLE design)
At the start: 16 parts

Commit message: Added initial version of ALU (Arithmetic Logic Unit) circuit
Parts:
- removed C3: 100nF, resistor:C-EU025-050X050
- removed C4: 10nF, resistor:C-EU025-050X050
- removed CLK1: NE555N, linear:NE555N
- removed DBG_BUTTON: (no value), switch-omron:10-XX
- removed LED2: (no value), eagle-ltspice:LED_ELD260
- added 4BIT-FULL-ADDER-0, 4BIT-FULL-ADDER-1: 74LS283N, 74xx-eu:74LS283N
- added DUAL-4X1-MUX-0, DUAL-4X1-MUX-1, DUAL-4X1-MUX-2, DUAL-4X1-MUX-3: 74LS153N, 74xx-eu:74LS153N
- added IC1, IC10, IC12, IC15, IC19, IC23, IC26, IC28, IC30, IC33, IC5, IC8: 74LS32N, 74xx-eu:74LS32N
- added IC11, IC14, IC16, IC21, IC22, IC25, IC27, IC29, IC3, IC32, IC4, IC7, IC9: 74LS08N, 74xx-eu:74LS08N
- added IC13, IC2, IC20, IC24, IC31, IC6: 74LS06N, 74xx-eu:74LS06N
- added IC17, IC18: 74LS86N, 74xx-eu:74LS86N
- added IC34: 74LS245N, 74xx-eu:74LS245N
- added Q1: BC556, transistor-pnp:BC556
- added Q2: BS170, transistor-small-signal:BS170
- added S1: (no value), switch-omron:10-XX
- added S2: 9077-1, switch-misc:9077-1
- R5: value 2.2k -> 1k
- R6: value 1k -> 10k
- R7: value 1M -> 10k
Connections:
- removed net CLK-Q: CLK.Q, LED1.C
- new net A: DUAL-4X1-MUX-0A.A, DUAL-4X1-MUX-1A.A, DUAL-4X1-MUX-2A.A, DUAL-4X1-MUX-3A.A, IC1A.I0
- new net ADD0-A0-IN: 4BIT-FULL-ADDER-0A.A1, IC17A.O, IC1D.I1, IC2B.I, IC3D.I0
- new net ADD0-A1-IN: 4BIT-FULL-ADDER-0A.A2, IC17B.O, IC2C.I, IC4A.I0, IC5A.I1
- new net ADD0-A2-IN: 4BIT-FULL-ADDER-0A.A3, IC17C.O, IC6B.I, IC7D.I0, IC8D.I1
- new net ADD0-A3-IN: 4BIT-FULL-ADDER-0A.A4, IC13B.I, IC14A.I0, IC15A.I1, IC17D.O
- new net ADD0-B0-IN: IC1D.I0, IC3D.I1
- new net ADD0-B1-IN: IC4A.I1, IC5A.I0
- new net ADD0-B2-IN: IC7D.I1, IC8D.I0
- new net ADD0-B3-IN: IC14A.I1, IC15A.I0
- new net ADD0-S0-OUT: 4BIT-FULL-ADDER-0A.S1, IC3B.I1
- new net ADD0-S1-OUT: 4BIT-FULL-ADDER-0A.S2, IC3C.I1
- new net ADD0-S2-OUT: 4BIT-FULL-ADDER-0A.S3, IC9B.I1
- new net ADD0-S3-OUT: 4BIT-FULL-ADDER-0A.S4, IC11C.I1
- new net ADD1-A4-IN: 4BIT-FULL-ADDER-1A.A1, IC18A.O, IC19D.I1, IC20B.I, IC21D.I0
- new net ADD1-A5-IN: 4BIT-FULL-ADDER-1A.A2, IC18B.O, IC20C.I, IC22A.I0, IC23A.I1
- new net ADD1-A6-IN: 4BIT-FULL-ADDER-1A.A3, IC18C.O, IC24B.I, IC25D.I0, IC26D.I1
- new net ADD1-A7-IN: 4BIT-FULL-ADDER-1A.A4, IC18D.O, IC31B.I, IC32A.I0, IC33A.I1
- new net ADD1-B4-IN: IC19D.I0, IC21D.I1
- new net ADD1-B5-IN: IC22A.I1, IC23A.I0
- new net ADD1-B6-IN: IC25D.I1, IC26D.I0
- new net ADD1-B7-IN: IC32A.I1, IC33A.I0
- new net ADD1-S4-OUT: 4BIT-FULL-ADDER-1A.S1, IC21B.I1
- new net ADD1-S5-OUT: 4BIT-FULL-ADDER-1A.S2, IC21C.I1
- new net ADD1-S6-OUT: 4BIT-FULL-ADDER-1A.S3, IC27B.I1
- new net ADD1-S7-OUT: 4BIT-FULL-ADDER-1A.S4, IC29C.I1
- new net ALU-A0-IN: IC17A.I1
- new net ALU-A1-IN: IC17B.I1
- new net ALU-A2-IN: IC17C.I1
- new net ALU-A3-IN: IC17D.I1
- new net ALU-A4-IN: IC18A.I1
- new net ALU-A5-IN: IC18B.I1
- new net ALU-A6-IN: IC18C.I1
- new net ALU-A7-IN: IC18D.I1
- new net ALU-B0-IN: 4BIT-FULL-ADDER-0A.B1
- new net ALU-B1-IN: 4BIT-FULL-ADDER-0A.B2
- new net ALU-B2-IN: 4BIT-FULL-ADDER-0A.B3
- new net ALU-B3-IN: 4BIT-FULL-ADDER-0A.B4
- new net ALU-B4-IN: 4BIT-FULL-ADDER-1A.B1
- new net ALU-B5-IN: 4BIT-FULL-ADDER-1A.B2
- new net ALU-B6-IN: 4BIT-FULL-ADDER-1A.B3
- new net ALU-B7-IN: 4BIT-FULL-ADDER-1A.B4
- new net ALU-C0-BUS-IN: IC34A.B1
- new net ALU-C0-OUT: IC1B.O, IC34A.A1
- new net ALU-C1-BUS-IN: IC34A.B2
- new net ALU-C1-OUT: IC1C.O, IC34A.A2
- new net ALU-C2-BUS-IN: IC34A.B3
- new net ALU-C2-OUT: IC10B.O, IC34A.A3
- new net ALU-C3-BUS-IN: IC34A.B4
- new net ALU-C3-OUT: IC12B.O, IC34A.A4
- new net ALU-C4-BUS-IN: IC34A.B5
- new net ALU-C4-OUT: IC19B.O, IC34A.A5
- new net ALU-C5-BUS-IN: IC34A.B6
- new net ALU-C5-OUT: IC19C.O, IC34A.A6
- new net ALU-C6-BUS-IN: IC34A.B7
- new net ALU-C6-OUT: IC28B.O, IC34A.A7
- new net ALU-C7-BUS-IN: IC34A.B8
- new net ALU-C7-OUT: IC30B.O, IC34A.A8
- new net ALU_EO: IC34A.G
- new net B: DUAL-4X1-MUX-0A.B, DUAL-4X1-MUX-1A.B, DUAL-4X1-MUX-2A.B, DUAL-4X1-MUX-3A.B, IC1A.I1
- new net C: 4BIT-FULL-ADDER-0A.C0, IC17A.I0, IC17B.I0, IC17C.I0, IC17D.I0, IC18A.I0, IC18B.I0, IC18C.I0, IC18D.I0
- new net CARRY-1: IC16A.O
- new net HLT: Q2.S, R7.1
- new net MUX-C0: IC11C.I0, IC16A.I0, IC21B.I0, IC21C.I0, IC29C.I0, IC2A.O, IC3A.I0, IC3B.I0, IC3C.I0
- new net MUX0-1C1-IN: DUAL-4X1-MUX-0A.1C1, IC1D.O
- new net MUX0-1C2-IN: DUAL-4X1-MUX-0A.1C2, IC2B.O
- new net MUX0-1C3-IN: DUAL-4X1-MUX-0A.1C3, IC3D.O
- new net MUX0-2C1-IN: DUAL-4X1-MUX-0A.2C1, IC5A.O
- new net MUX0-2C2-IN: DUAL-4X1-MUX-0A.2C2, IC2C.O
- new net MUX0-2C3-IN: DUAL-4X1-MUX-0A.2C3, IC4A.O
- new net MUX0-C0: IC27B.I0, IC9B.I0
- new net MUX1-1C1-IN: DUAL-4X1-MUX-1A.1C1, IC8D.O
- new net MUX1-1C2-IN: DUAL-4X1-MUX-1A.1C2, IC6B.O
- new net MUX1-1C3-IN: DUAL-4X1-MUX-1A.1C3, IC7D.O
- new net MUX1-2C1-IN: DUAL-4X1-MUX-1A.2C1, IC15A.O
- new net MUX1-2C2-IN: DUAL-4X1-MUX-1A.2C2, IC13B.O
- new net MUX1-2C3-IN: DUAL-4X1-MUX-1A.2C3, IC14A.O
- new net MUX2-1C1-IN: DUAL-4X1-MUX-2A.1C1, IC19D.O
- new net MUX2-1C2-IN: DUAL-4X1-MUX-2A.1C2, IC20B.O
- new net MUX2-1C3-IN: DUAL-4X1-MUX-2A.1C3, IC21D.O
- new net MUX2-2C1-IN: DUAL-4X1-MUX-2A.2C1, IC23A.O
- new net MUX2-2C2-IN: DUAL-4X1-MUX-2A.2C2, IC20C.O
- new net MUX2-2C3-IN: DUAL-4X1-MUX-2A.2C3, IC22A.O
- new net MUX3-1C1-IN: DUAL-4X1-MUX-3A.1C1, IC26D.O
- new net MUX3-1C2-IN: DUAL-4X1-MUX-3A.1C2, IC24B.O
- new net MUX3-1C3-IN: DUAL-4X1-MUX-3A.1C3, IC25D.O
- new net MUX4-2C1-IN: DUAL-4X1-MUX-3A.2C1, IC33A.O
- new net MUX4-2C2-IN: DUAL-4X1-MUX-3A.2C2, IC31B.O
- new net MUX4-2C3-IN: DUAL-4X1-MUX-3A.2C3, IC32A.O
- new net N$10: IC10B.I0, IC9B.O
- new net N$11: DUAL-4X1-MUX-1A.1Y, IC10B.I1
- new net N$12: DUAL-4X1-MUX-1A.2Y, IC12B.I0
- new net N$13: DUAL-4X1-MUX-0A.1Y, IC1B.I1
- new net N$14: IC1C.I1, IC3C.O
- new net N$15: IC11C.O, IC12B.I1
- new net N$16: 4BIT-FULL-ADDER-1A.C0, IC3A.O
- new net N$18: DUAL-4X1-MUX-2A.1Y, IC19B.I1
- new net N$19: DUAL-4X1-MUX-2A.2Y, IC19C.I0
- new net N$20: IC19C.I1, IC21C.O
- new net N$21: IC27B.O, IC28B.I0
- new net N$22: DUAL-4X1-MUX-3A.1Y, IC28B.I1
- new net N$23: DUAL-4X1-MUX-3A.2Y, IC30B.I0
- new net N$24: IC29C.O, IC30B.I1
- new net N$8: DUAL-4X1-MUX-0A.2Y, IC1C.I0
- new net N$9: 4BIT-FULL-ADDER-1A.C4, IC16A.I1
- new net Q: CLK.Q, Q2.G, R7.2
- new net S0_1_OUT: IC1B.I0, IC3B.O
- new net S0_1_OUT1: IC19B.I0, IC21B.O
- net CLK-DIS: now also Q1.C; no longer R1.1
- net CLK-TR-THR: now also Q1.B, R6.1, R6.2, S2.S
- net GND: now also DUAL-4X1-MUX-0A.1C0, DUAL-4X1-MUX-0A.2C0, DUAL-4X1-MUX-1A.1C0, DUAL-4X1-MUX-1A.2C0, DUAL-4X1-MUX-2A.1C0, DUAL-4X1-MUX-2A.2C0, DUAL-4X1-MUX-3A.1C0, DUAL-4X1-MUX-3A.2C0, S1.S, S2.O, S2.P; no longer C3.1, C4.2, CLK1.GND, DBG_BUTTON.P1, R5.2
- net N$1: now also R5.1, S1.P; no longer CLK1.Q, LED2.C
- net N$3: now also CLK.V+, Q1.E, R1.1; no longer LED2.A, R5.1
- net N$4: now also LED1.C; no longer LED1.A
- net N$5: now also IC1A.O, IC2A.I; no longer CLK1.TR, DBG_BUTTON.S1, R6.1
- net N$6: now also LED1.A, Q2.D; no longer C3.2, CLK1.DIS, CLK1.THR, R7.1
- net N$7: now also 4BIT-FULL-ADDER-0A.C4, IC3A.I1; no longer C4.1, CLK1.CV
- net VCC: now also DUAL-4X1-MUX-0A.1G, DUAL-4X1-MUX-0A.2G, DUAL-4X1-MUX-1A.1G, DUAL-4X1-MUX-1A.2G, DUAL-4X1-MUX-2A.1G, DUAL-4X1-MUX-2A.2G, DUAL-4X1-MUX-3A.1G, DUAL-4X1-MUX-3A.2G, IC34A.DIR, R5.2; no longer CLK.V+, CLK1.R, CLK1.V+, R6.2, R7.2
Other:
- note added: "8-BIT COMPUTER"
- note added: "ALU (ARITHMETIC LOGIC UNIT)"
- note added: "MAIN CLK"
- note removed: "MAIN CLK - ASTABLE MODE"
- note removed: "STEPPING CLK - MONOSTABLE MODE"
- moved on the sheet: C1, C2, CLK, LED1, R1, R2, R3, R4, R5, R6, R7

Commit message: Added fixes for ALU schema
Connections:
- removed net ADD0-B0-IN: IC1D.I0, IC3D.I1
- removed net ADD0-B1-IN: IC4A.I1, IC5A.I0
- removed net ADD0-B2-IN: IC7D.I1, IC8D.I0
- removed net ADD0-B3-IN: IC14A.I1, IC15A.I0
- removed net ADD1-B4-IN: IC19D.I0, IC21D.I1
- removed net ADD1-B5-IN: IC22A.I1, IC23A.I0
- removed net ADD1-B6-IN: IC25D.I1, IC26D.I0
- removed net ADD1-B7-IN: IC32A.I1, IC33A.I0
- net ADD0-A0-IN: no longer IC1D.I1, IC2B.I, IC3D.I0
- net ADD0-A1-IN: no longer IC2C.I, IC4A.I0, IC5A.I1
- net ADD0-A2-IN: no longer IC6B.I, IC7D.I0, IC8D.I1
- net ADD0-A3-IN: no longer IC13B.I, IC14A.I0, IC15A.I1
- net ADD1-A4-IN: no longer IC19D.I1, IC20B.I, IC21D.I0
- net ADD1-A5-IN: no longer IC20C.I, IC22A.I0, IC23A.I1
- net ADD1-A6-IN: no longer IC24B.I, IC25D.I0, IC26D.I1
- net ADD1-A7-IN: no longer IC31B.I, IC32A.I0, IC33A.I1
- net ALU-A0-IN: now also IC1D.I1, IC2B.I, IC3D.I0
- net ALU-A1-IN: now also IC2C.I, IC4A.I0, IC5A.I1
- net ALU-A2-IN: now also IC6B.I, IC7D.I0, IC8D.I1
- net ALU-A3-IN: now also IC13B.I, IC14A.I0, IC15A.I1
- net ALU-A4-IN: now also IC19D.I1, IC20B.I, IC21D.I0
- net ALU-A5-IN: now also IC20C.I, IC22A.I0, IC23A.I1
- net ALU-A6-IN: now also IC24B.I, IC25D.I0, IC26D.I1
- net ALU-A7-IN: now also IC31B.I, IC32A.I0, IC33A.I1
- net ALU-B0-IN: now also IC1D.I0, IC3D.I1
- net ALU-B1-IN: now also IC4A.I1, IC5A.I0
- net ALU-B2-IN: now also IC7D.I1, IC8D.I0
- net ALU-B3-IN: now also IC14A.I1, IC15A.I0
- net ALU-B4-IN: now also IC19D.I0, IC21D.I1
- net ALU-B5-IN: now also IC22A.I1, IC23A.I0
- net ALU-B6-IN: now also IC25D.I1, IC26D.I0
- net ALU-B7-IN: now also IC32A.I1, IC33A.I0
- net GND: now also DUAL-4X1-MUX-0A.1G, DUAL-4X1-MUX-0A.2G, DUAL-4X1-MUX-1A.1G, DUAL-4X1-MUX-1A.2G, DUAL-4X1-MUX-2A.1G, DUAL-4X1-MUX-2A.2G, DUAL-4X1-MUX-3A.1G, DUAL-4X1-MUX-3A.2G
- net VCC: no longer DUAL-4X1-MUX-0A.1G, DUAL-4X1-MUX-0A.2G, DUAL-4X1-MUX-1A.1G, DUAL-4X1-MUX-1A.2G, DUAL-4X1-MUX-2A.1G, DUAL-4X1-MUX-2A.2G, DUAL-4X1-MUX-3A.1G, DUAL-4X1-MUX-3A.2G

Commit message: Changed 74LS06N which is inverter with open collector outputs into 74LS04N with standard outputs
Parts:
- removed IC20, IC24, IC31: 74LS06N, 74xx-eu:74LS06N
- removed IC27, IC29: 74LS08N, 74xx-eu:74LS08N
- removed IC28, IC30: 74LS32N, 74xx-eu:74LS32N
- IC10, IC12: value 74LS32N -> 74LS04N; device 74xx-eu:74LS32N -> 74xx-eu:74LS04N
- IC11, IC16, IC9: value 74LS08N -> 74LS04N; device 74xx-eu:74LS08N -> 74xx-eu:74LS04N
- IC13, IC2, IC6: value 74LS06N -> 74LS04N; device 74xx-eu:74LS06N -> 74xx-eu:74LS04N
Connections:
- removed net ADD0-S0-OUT: 4BIT-FULL-ADDER-0A.S1, IC3B.I1
- removed net ADD0-S1-OUT: 4BIT-FULL-ADDER-0A.S2, IC3C.I1
- removed net ADD0-S2-OUT: 4BIT-FULL-ADDER-0A.S3, IC9B.I1
- removed net ADD0-S3-OUT: 4BIT-FULL-ADDER-0A.S4, IC11C.I1
- removed net ADD1-S4-OUT: 4BIT-FULL-ADDER-1A.S1, IC21B.I1
- removed net ADD1-S5-OUT: 4BIT-FULL-ADDER-1A.S2, IC21C.I1
- removed net ADD1-S6-OUT: 4BIT-FULL-ADDER-1A.S3, IC27B.I1
- removed net ADD1-S7-OUT: 4BIT-FULL-ADDER-1A.S4, IC29C.I1
- removed net MUX-C0: IC11C.I0, IC16A.I0, IC21B.I0, IC21C.I0, IC29C.I0, IC2A.O, IC3A.I0, IC3B.I0, IC3C.I0
- removed net MUX0-C0: IC27B.I0, IC9B.I0
- removed net N$10: IC10B.I0, IC9B.O
- removed net N$11: DUAL-4X1-MUX-1A.1Y, IC10B.I1
- removed net N$12: DUAL-4X1-MUX-1A.2Y, IC12B.I0
- removed net N$13: DUAL-4X1-MUX-0A.1Y, IC1B.I1
- removed net N$14: IC1C.I1, IC3C.O
- removed net N$15: IC11C.O, IC12B.I1
- removed net N$16: 4BIT-FULL-ADDER-1A.C0, IC3A.O
- removed net N$18: DUAL-4X1-MUX-2A.1Y, IC19B.I1
- removed net N$19: DUAL-4X1-MUX-2A.2Y, IC19C.I0
- removed net N$20: IC19C.I1, IC21C.O
- removed net N$21: IC27B.O, IC28B.I0
- removed net N$22: DUAL-4X1-MUX-3A.1Y, IC28B.I1
- removed net N$23: DUAL-4X1-MUX-3A.2Y, IC30B.I0
- removed net N$24: IC29C.O, IC30B.I1
- removed net N$7: 4BIT-FULL-ADDER-0A.C4, IC3A.I1
- removed net N$8: DUAL-4X1-MUX-0A.2Y, IC1C.I0
- removed net N$9: 4BIT-FULL-ADDER-1A.C4, IC16A.I1
- removed net S0_1_OUT: IC1B.I0, IC3B.O
- removed net S0_1_OUT1: IC19B.I0, IC21B.O
- new net MUX0-1C0-IN: 4BIT-FULL-ADDER-0A.S1, DUAL-4X1-MUX-0A.1C0
- new net MUX0-2C0-IN: 4BIT-FULL-ADDER-0A.S2, DUAL-4X1-MUX-0A.2C0
- new net MUX1-1C0-IN: 4BIT-FULL-ADDER-0A.S3, DUAL-4X1-MUX-1A.1C0
- new net MUX1-2C0-IN: 4BIT-FULL-ADDER-0A.S4, DUAL-4X1-MUX-1A.2C0
- new net MUX2-1C0-IN: 4BIT-FULL-ADDER-1A.S1, DUAL-4X1-MUX-2A.1C0
- new net MUX2-2C0-IN: 4BIT-FULL-ADDER-1A.S2, DUAL-4X1-MUX-2A.2C0
- new net MUX3-1C0-IN: 4BIT-FULL-ADDER-1A.S3, DUAL-4X1-MUX-3A.1C0
- new net MUX3-2C0-IN: 4BIT-FULL-ADDER-1A.S4, DUAL-4X1-MUX-3A.2C0
- net A: no longer IC1A.I0
- net ALU-A0-IN: now also IC9A.I; no longer IC2B.I
- net ALU-A1-IN: now also IC2A.I; no longer IC2C.I
- net ALU-A2-IN: now also IC6A.I; no longer IC6B.I
- net ALU-A3-IN: now also IC10A.I; no longer IC13B.I
- net ALU-A4-IN: now also IC11A.I; no longer IC20B.I
- net ALU-A5-IN: now also IC12A.I; no longer IC20C.I
- net ALU-A6-IN: now also IC13A.I; no longer IC24B.I
- net ALU-A7-IN: now also IC16A.I; no longer IC31B.I
- net ALU-C0-OUT: now also DUAL-4X1-MUX-0A.1Y; no longer IC1B.O
- net ALU-C1-OUT: now also DUAL-4X1-MUX-0A.2Y; no longer IC1C.O
- net ALU-C2-OUT: now also DUAL-4X1-MUX-1A.1Y; no longer IC10B.O
- net ALU-C3-OUT: now also DUAL-4X1-MUX-1A.2Y; no longer IC12B.O
- net ALU-C4-OUT: now also DUAL-4X1-MUX-2A.1Y; no longer IC19B.O
- net ALU-C5-OUT: now also DUAL-4X1-MUX-2A.2Y; no longer IC19C.O
- net ALU-C6-OUT: now also DUAL-4X1-MUX-3A.1Y; no longer IC28B.O
- net ALU-C7-OUT: now also DUAL-4X1-MUX-3A.2Y; no longer IC30B.O
- net B: no longer IC1A.I1
- net CARRY-1: now also 4BIT-FULL-ADDER-1A.C4; no longer IC16A.O
- net GND: no longer DUAL-4X1-MUX-0A.1C0, DUAL-4X1-MUX-0A.2C0, DUAL-4X1-MUX-1A.1C0, DUAL-4X1-MUX-1A.2C0, DUAL-4X1-MUX-2A.1C0, DUAL-4X1-MUX-2A.2C0, DUAL-4X1-MUX-3A.1C0, DUAL-4X1-MUX-3A.2C0
- net MUX0-1C2-IN: now also IC9A.O; no longer IC2B.O
- net MUX0-2C2-IN: now also IC2A.O; no longer IC2C.O
- net MUX1-1C2-IN: now also IC6A.O; no longer IC6B.O
- net MUX1-2C2-IN: now also IC10A.O; no longer IC13B.O
- net MUX2-1C2-IN: now also IC11A.O; no longer IC20B.O
- net MUX2-2C2-IN: now also IC12A.O; no longer IC20C.O
- net MUX3-1C2-IN: now also IC13A.O; no longer IC24B.O
- net MUX4-2C2-IN: now also IC16A.O; no longer IC31B.O
- net N$5: now also 4BIT-FULL-ADDER-0A.C4, 4BIT-FULL-ADDER-1A.C0; no longer IC1A.O, IC2A.I
Other:
- moved on the sheet: 4BIT-FULL-ADDER-1, IC16A, IC2A, IC34
