File: rel-8bit-computer.sch (EAGLE design)
At the start: 57 parts, among them IC1 74LS04N, IC2 74LS04N, IC3 74LS04N, IC35 74LS32N, IC37 74LS08N, IC38 74LS08N, IC39 74LS32N, IC4 74LS04N, IC41 74LS08N, IC42 74LS32N, IC44 74LS08N, IC45 74LS32N, IC46 74LS86N, IC47 74LS86N, IC48 74LS32N, IC5 74LS04N, IC50 74LS08N, IC51 74LS08N, IC52 74LS32N, IC54 74LS08N, IC55 74LS32N, IC57 74LS08N, IC58 74LS32N, IC59 74LS245N, IC6 74LS04N, IC7 74LS04N, IC8 74LS04N, Q1 BC556, Q2 BS170

Commit message: Added initial schema for general purpose registers
Parts:
- removed PAGE-ADD-REG-1, PAGE-ADDR-REG-2, PAGE-ADDR-REG-3: 74LS173N, 74xx-eu:74LS173N
- added ADDR-R/P-SW-0, ADDR-R/P-SW-1, ADDR-R/P-SW-2, ADDR-R/P-SW-3, DATA-R/P-SW-0, DATA-R/P-SW-1: 74LS157N, 74xx-eu:74LS157N
- added BUFFER-0, BUFFER-1, BUFFER-2, BUFFER-3, IC17, IC18: 74LS245N, 74xx-eu:74LS245N
- added C3, C4: 2n, resistor:C-EU025-025X050
- added D1, D2, D3, D4: (no value), special:7SEG-CK
- added IC10: (no value), memory:2816
- added IC11: NE555N, linear:NE555N
- added IC12: 74LS139N, 74xx-eu:74LS139N
- added IC13, IC14, IC15, IC16: 74160N, 74xx-eu:74160N
- added IC19: 74LS04N, 74xx-eu:74LS04N
- added IC9: 7476N, 74xx-eu:7476N
- added LED10, LED11, LED12, LED13, LED14, LED15, LED16, LED17, LED18, LED19, LED2, LED20, LED21, LED22, LED23, LED24, LED25, LED26, LED3, LED4, LED5, LED6, LED7, LED8, LED9: (no value), led:LED5MM
- added PROG/RUN-ADDR-SW: (no value), special:SW_DIP-12
- added PROG/RUN-DATA-SW: (no value), special:SW_DIP-8
- added R8: 100k, resistor:R-EU_0204/5
- added R9: 1k, resistor:R-EU_0204/5
- added SW2, SW3: (no value), special:SW_DIP-1
Connections:
- removed net DATA0: MEMORY-0-8KX8-6264.I/O1, MEMORY-1-8KX8-6264.I/O1, MEMORY-2-8KX8-6264.I/O1, MEMORY-3-8KX8-6264.I/O1, PAGE-ADD-REG-1A.D1, PAGE-ADDR-REG-0A.D1, PAGE-ADDR-REG-2A.D1, PAGE-ADDR-REG-3A.D1
- removed net DATA1: MEMORY-0-8KX8-6264.I/O2, MEMORY-1-8KX8-6264.I/O2, MEMORY-2-8KX8-6264.I/O2, MEMORY-3-8KX8-6264.I/O2, PAGE-ADD-REG-1A.D2, PAGE-ADDR-REG-0A.D2, PAGE-ADDR-REG-2A.D2, PAGE-ADDR-REG-3A.D2
- removed net DATA2: MEMORY-0-8KX8-6264.I/O3, MEMORY-1-8KX8-6264.I/O3, MEMORY-2-8KX8-6264.I/O3, MEMORY-3-8KX8-6264.I/O3, PAGE-ADD-REG-1A.D3, PAGE-ADDR-REG-0A.D3, PAGE-ADDR-REG-2A.D3, PAGE-ADDR-REG-3A.D3
- removed net DATA3: MEMORY-0-8KX8-6264.I/O4, MEMORY-1-8KX8-6264.I/O4, MEMORY-2-8KX8-6264.I/O4, MEMORY-3-8KX8-6264.I/O4, PAGE-ADD-REG-1A.D4, PAGE-ADDR-REG-2A.D4, PAGE-ADDR-REG-3A.D4
- removed net DATA4: MEMORY-0-8KX8-6264.I/O5, MEMORY-1-8KX8-6264.I/O5, MEMORY-2-8KX8-6264.I/O5, MEMORY-3-8KX8-6264.I/O5, PAGE-ADDR-REG-0A.D4
- removed net DATA5: MEMORY-0-8KX8-6264.I/O6, MEMORY-1-8KX8-6264.I/O6, MEMORY-2-8KX8-6264.I/O6, MEMORY-3-8KX8-6264.I/O6
- removed net DATA6: MEMORY-0-8KX8-6264.I/O7, MEMORY-1-8KX8-6264.I/O7, MEMORY-2-8KX8-6264.I/O7, MEMORY-3-8KX8-6264.I/O7
- removed net DATA7: MEMORY-0-8KX8-6264.I/O8, MEMORY-1-8KX8-6264.I/O8, MEMORY-2-8KX8-6264.I/O8, MEMORY-3-8KX8-6264.I/O8
- removed net PAGE-EN-2: MEMORY-2-8KX8-6264.!CS1
- removed net PAGE-EN0: DEMUX-2X4-0A.Y0, MEMORY-0-8KX8-6264.!CS1, PAGE-ADDR-REG-0A.G1, PAGE-ADDR-REG-0A.G2
- removed net PAGE-EN1: DEMUX-2X4-0A.Y1, MEMORY-1-8KX8-6264.!CS1, PAGE-ADD-REG-1A.G1, PAGE-ADD-REG-1A.G2
- removed net PAGE-EN2: DEMUX-2X4-0A.Y2, PAGE-ADDR-REG-2A.G1, PAGE-ADDR-REG-2A.G2
- removed net PAGE-EN3: DEMUX-2X4-0A.Y3, MEMORY-3-8KX8-6264.!CS1, PAGE-ADDR-REG-3A.G1, PAGE-ADDR-REG-3A.G2
- new net ADDR-A12: ADDR-R/P-SW-3A.1Y, BUFFER-3A.A1, LED26.A
- new net ADDR-B0: BUFFER-0A.B5, MEMORY-0-8KX8-6264.A0, MEMORY-1-8KX8-6264.A0, MEMORY-2-8KX8-6264.A0, MEMORY-3-8KX8-6264.A0
- new net ADDR-B1: BUFFER-0A.B6, MEMORY-0-8KX8-6264.A1, MEMORY-1-8KX8-6264.A1, MEMORY-2-8KX8-6264.A1, MEMORY-3-8KX8-6264.A1
- new net ADDR-B2: BUFFER-0A.B7, MEMORY-0-8KX8-6264.A2, MEMORY-1-8KX8-6264.A2, MEMORY-2-8KX8-6264.A2, MEMORY-3-8KX8-6264.A2
- new net ADDR-B3: BUFFER-0A.B8, MEMORY-0-8KX8-6264.A3, MEMORY-1-8KX8-6264.A3, MEMORY-2-8KX8-6264.A3, MEMORY-3-8KX8-6264.A3
- new net ADDR-B4: BUFFER-1A.B1, MEMORY-0-8KX8-6264.A4, MEMORY-1-8KX8-6264.A4, MEMORY-2-8KX8-6264.A4, MEMORY-3-8KX8-6264.A4
- new net ADDR-B5: BUFFER-1A.B2, MEMORY-0-8KX8-6264.A5, MEMORY-1-8KX8-6264.A5, MEMORY-2-8KX8-6264.A5, MEMORY-3-8KX8-6264.A5
- new net ADDR-B6: BUFFER-1A.B3, MEMORY-0-8KX8-6264.A6, MEMORY-1-8KX8-6264.A6, MEMORY-2-8KX8-6264.A6, MEMORY-3-8KX8-6264.A6
- new net ADDR-B7: BUFFER-1A.B4, MEMORY-0-8KX8-6264.A7, MEMORY-1-8KX8-6264.A7, MEMORY-2-8KX8-6264.A7, MEMORY-2-8KX8-6264.A8, MEMORY-3-8KX8-6264.A7
- new net ADDR-B8: BUFFER-1A.B5, MEMORY-0-8KX8-6264.A8, MEMORY-1-8KX8-6264.A8, MEMORY-3-8KX8-6264.A8
- new net ADDR-B9: BUFFER-1A.B6, MEMORY-0-8KX8-6264.A9, MEMORY-1-8KX8-6264.A9, MEMORY-2-8KX8-6264.A9, MEMORY-3-8KX8-6264.A9
- new net ADDR-BUS0: ADDR-R/P-SW-0A.1A, IC13A.A
- new net ADDR-BUS1: ADDR-R/P-SW-0A.2A, IC13A.B
- new net ADDR-BUS10: DEMUX-2X4-0A.B
- new net ADDR-BUS2: ADDR-R/P-SW-0A.3A, IC13A.C
- new net ADDR-BUS3: ADDR-R/P-SW-0A.4A, IC13A.D
- new net ADDR-BUS4: ADDR-R/P-SW-1A.1A, IC14A.A
- new net ADDR-BUS5: ADDR-R/P-SW-1A.2A, IC14A.B
- new net ADDR-BUS6: ADDR-R/P-SW-1A.3A, IC14A.C
- new net ADDR-BUS7: ADDR-R/P-SW-1A.4A, IC14A.D
- new net ADDR-BUS8: ADDR-R/P-SW-2A.1A, IC15A.A
- new net ADDR-BUS9: DEMUX-2X4-0A.A
- new net ADDR-PAGE10: ADDR-R/P-SW-2A.3A, IC15A.C, PAGE-ADDR-REG-0A.Q2
- new net ADDR-PAGE11: ADDR-R/P-SW-2A.4A, IC15A.D, PAGE-ADDR-REG-0A.Q3
- new net ADDR-PAGE12: ADDR-R/P-SW-3A.1A, IC16A.A, PAGE-ADDR-REG-0A.Q4
- new net ADDR-PAGE9: ADDR-R/P-SW-2A.2A, IC15A.B, PAGE-ADDR-REG-0A.Q1
- new net ADDR-PROG0: ADDR-R/P-SW-0A.1B, PROG/RUN-ADDR-SW.1
- new net ADDR-PROG1: ADDR-R/P-SW-0A.2B, PROG/RUN-ADDR-SW.2
- new net ADDR-PROG10: ADDR-R/P-SW-2A.3B, PROG/RUN-ADDR-SW.11
- new net ADDR-PROG11: ADDR-R/P-SW-2A.4B, PROG/RUN-ADDR-SW.12
- new net ADDR-PROG12: ADDR-R/P-SW-3A.1B, SW3.1
- new net ADDR-PROG2: ADDR-R/P-SW-0A.3B, PROG/RUN-ADDR-SW.3
- new net ADDR-PROG3: ADDR-R/P-SW-0A.4B, PROG/RUN-ADDR-SW.4
- new net ADDR-PROG4: ADDR-R/P-SW-1A.1B, PROG/RUN-ADDR-SW.5
- new net ADDR-PROG5: ADDR-R/P-SW-1A.2B, PROG/RUN-ADDR-SW.6
- new net ADDR-PROG6: ADDR-R/P-SW-1A.3B, PROG/RUN-ADDR-SW.7
- new net ADDR-PROG7: ADDR-R/P-SW-1A.4B, PROG/RUN-ADDR-SW.8
- new net ADDR-PROG8: ADDR-R/P-SW-2A.1B, PROG/RUN-ADDR-SW.9
- new net ADDR-PROG9: ADDR-R/P-SW-2A.2B, PROG/RUN-ADDR-SW.10
- new net COUNTER-CARRY-0: IC13A.RCO, IC14A.ENT
- new net COUNTER-CARRY-1: IC14A.RCO, IC15A.ENT
- new net COUNTER-CARRY-2: IC15A.RCO, IC16A.ENT
- new net COUNTER-EN: IC13A.ENP, IC13A.ENT, IC14A.ENP, IC15A.ENP, IC16A.ENP
- new net COUNTER-OUT: IC17A.G, IC18A.G
- new net COUNTER-RST: IC13A.CLR, IC14A.CLR, IC15A.CLR, IC16A.CLR, IC19A.O
- new net DATA-A0: BUFFER-2A.B1, DATA-R/P-SW-0A.1Y, IC18A.B2, PAGE-ADDR-REG-0A.D1
- new net DATA-A1: BUFFER-2A.B2, DATA-R/P-SW-0A.2Y, IC18A.B3, PAGE-ADDR-REG-0A.D2
- new net DATA-A2: BUFFER-2A.B3, DATA-R/P-SW-0A.3Y, IC18A.B4, PAGE-ADDR-REG-0A.D3
- new net DATA-A3: BUFFER-2A.B4, DATA-R/P-SW-0A.4Y, IC18A.B5, PAGE-ADDR-REG-0A.D4
- new net DATA-A4: BUFFER-2A.B5, DATA-R/P-SW-1A.1Y
- new net DATA-A5: BUFFER-2A.B6, DATA-R/P-SW-1A.2Y
- new net DATA-A6: BUFFER-2A.B7, DATA-R/P-SW-1A.3Y
- new net DATA-A7: BUFFER-2A.B8, DATA-R/P-SW-1A.4Y
- new net DATA-B0: BUFFER-2A.A1, LED25.A, MEMORY-0-8KX8-6264.I/O1, MEMORY-1-8KX8-6264.I/O1, MEMORY-2-8KX8-6264.I/O1, MEMORY-3-8KX8-6264.I/O1
- new net DATA-B1: BUFFER-2A.A2, LED24.A, MEMORY-0-8KX8-6264.I/O2, MEMORY-1-8KX8-6264.I/O2, MEMORY-2-8KX8-6264.I/O2, MEMORY-3-8KX8-6264.I/O2
- new net DATA-B2: BUFFER-2A.A3, LED23.A, MEMORY-0-8KX8-6264.I/O3, MEMORY-1-8KX8-6264.I/O3, MEMORY-2-8KX8-6264.I/O3, MEMORY-3-8KX8-6264.I/O3
- new net DATA-B3: BUFFER-2A.A4, LED22.A, MEMORY-0-8KX8-6264.I/O4, MEMORY-1-8KX8-6264.I/O4, MEMORY-2-8KX8-6264.I/O4, MEMORY-3-8KX8-6264.I/O4
- new net DATA-B4: BUFFER-2A.A5, LED21.A, MEMORY-0-8KX8-6264.I/O5, MEMORY-1-8KX8-6264.I/O5, MEMORY-2-8KX8-6264.I/O5, MEMORY-3-8KX8-6264.I/O5
- new net DATA-B5: BUFFER-2A.A6, LED20.A, MEMORY-0-8KX8-6264.I/O6, MEMORY-1-8KX8-6264.I/O6, MEMORY-2-8KX8-6264.I/O6, MEMORY-3-8KX8-6264.I/O6
- new net DATA-B6: BUFFER-2A.A7, LED19.A, MEMORY-0-8KX8-6264.I/O7, MEMORY-1-8KX8-6264.I/O7, MEMORY-2-8KX8-6264.I/O7, MEMORY-3-8KX8-6264.I/O7
- new net DATA-B7: BUFFER-2A.A8, LED18.A, MEMORY-0-8KX8-6264.I/O8, MEMORY-1-8KX8-6264.I/O8, MEMORY-2-8KX8-6264.I/O8, MEMORY-3-8KX8-6264.I/O8
- new net DATA-BUS0: DATA-R/P-SW-0A.1A, IC17A.B1
- new net DATA-BUS1: DATA-R/P-SW-0A.2A, IC17A.B2
- new net DATA-BUS2: DATA-R/P-SW-0A.3A, IC17A.B3
- new net DATA-BUS3: DATA-R/P-SW-0A.4A, IC17A.B4
- new net DATA-BUS4: DATA-R/P-SW-1A.1A, IC17A.B5
- new net DATA-BUS5: DATA-R/P-SW-1A.2A, IC17A.B6
- new net DATA-BUS6: DATA-R/P-SW-1A.3A, IC17A.B7
- new net DATA-BUS7: DATA-R/P-SW-1A.4A, IC17A.B8
- new net DATA-BUS8: IC18A.B1
- new net DATA-OUT0: IC13A.QA, IC17A.A1
- new net DATA-OUT1: IC13A.QB, IC17A.A2
- new net DATA-OUT10: IC15A.QC, IC18A.A3
- new net DATA-OUT11: IC15A.QD, IC18A.A4
- new net DATA-OUT12: IC16A.QA, IC18A.A5
- new net DATA-OUT2: IC13A.QC, IC17A.A3
- new net DATA-OUT3: IC13A.QD, IC17A.A4
- new net DATA-OUT4: IC14A.QA, IC17A.A5
- new net DATA-OUT5: IC14A.QB, IC17A.A6
- new net DATA-OUT6: IC14A.QC, IC17A.A7
- new net DATA-OUT7: IC14A.QD, IC17A.A8
- new net DATA-OUT8: IC15A.QA, IC18A.A1
- new net DATA-OUT9: IC15A.QB, IC18A.A2
- new net DATA-PROG0: DATA-R/P-SW-0A.1B, PROG/RUN-DATA-SW.1
- new net DATA-PROG1: DATA-R/P-SW-0A.2B, PROG/RUN-DATA-SW.2
- new net DATA-PROG2: DATA-R/P-SW-0A.3B, PROG/RUN-DATA-SW.3
- new net DATA-PROG3: DATA-R/P-SW-0A.4B, PROG/RUN-DATA-SW.4
- new net DATA-PROG4: DATA-R/P-SW-1A.1B, PROG/RUN-DATA-SW.5
- new net DATA-PROG5: DATA-R/P-SW-1A.2B, PROG/RUN-DATA-SW.6
- new net DATA-PROG6: DATA-R/P-SW-1A.3B, PROG/RUN-DATA-SW.7
- new net DATA-PROG7: DATA-R/P-SW-1A.4B, PROG/RUN-DATA-SW.8
- new net DISP-CLK: IC11.Q, IC9A.CLK
- new net DISP-DATA-IN0: IC10A.A0
- new net DISP-DATA-IN1: IC10A.A1
- new net DISP-DATA-IN2: IC10A.A2
- new net DISP-DATA-IN3: IC10A.A3
- new net DISP-DATA-IN4: IC10A.A4
- new net DISP-DATA-IN5: IC10A.A5
- new net DISP-DATA-IN6: IC10A.A6
- new net DISP-DATA-IN7: IC10A.A7
- new net DISP-DATA-OUT0: D1.A, D2.A, D3.A, D4.A, IC10A.D0
- new net DISP-DATA-OUT1: D1.B, D2.B, D3.B, D4.B, IC10A.D1
- new net DISP-DATA-OUT2: D1.C, D2.C, D3.C, D4.C, IC10A.D2
- new net DISP-DATA-OUT3: D1.D, D2.D, D3.D, D4.D, IC10A.D3
- new net DISP-DATA-OUT4: D1.E, D2.E, D3.E, D4.E, IC10A.D4
- new net DISP-DATA-OUT5: D1.F, D2.F, D3.F, D4.F, IC10A.D5
- new net DISP-DATA-OUT6: D1.G, D2.G, D3.G, D4.G, IC10A.D6
- new net DISP-DATA-OUT7: D1.DP, D2.DP, D3.DP, D4.DP, IC10A.D7
- new net DISP-EN0: D1.CK1, D1.CK2, IC12A.Y0
- new net DISP-EN1: D2.CK1, D2.CK2, IC12A.Y1
- new net DISP-EN2: D3.CK1, D3.CK2, IC12A.Y2
- new net DISP-EN3: D4.CK1, D4.CK2, IC12A.Y3
- new net DISP-FF-OUT0: IC10A.A8, IC12A.A, IC9A.Q, IC9B.CLK
- new net DISP-FF-OUT1: IC10A.A9, IC12A.B, IC9B.Q
- new net DISP-NEG-SWITCH: IC10A.A10
- new net DISP-TRIG: C4.2, IC11.THR, IC11.TR, R8.2, R9.2
- new net JMP-SIG: IC13A.LD, IC14A.LD, IC15A.LD, IC16A.LD
- new net N$7: C3.1, IC11.CV
- new net N$8: IC11.DIS, R8.1
- new net N$9: IC16A.QB, IC19A.I
- new net PAGE-EN-A0: BUFFER-0A.A1, DEMUX-2X4-0A.Y0, LED12.A
- new net PAGE-EN-A1: BUFFER-0A.A2, DEMUX-2X4-0A.Y1, LED13.A
- new net PAGE-EN-A2: BUFFER-0A.A3, DEMUX-2X4-0A.Y2, LED14.A
- new net PAGE-EN-A3: BUFFER-0A.A4, DEMUX-2X4-0A.Y3, LED15.A
- new net PAGE-EN-B0: BUFFER-0A.B1, MEMORY-0-8KX8-6264.!CS1
- new net PAGE-EN-B1: BUFFER-0A.B2, MEMORY-1-8KX8-6264.!CS1
- new net PAGE-EN-B2: BUFFER-0A.B3, MEMORY-2-8KX8-6264.!CS1
- new net PAGE-EN-B3: BUFFER-0A.B4, MEMORY-3-8KX8-6264.!CS1
- new net PR-LOAD: PAGE-ADDR-REG-0A.G1, PAGE-ADDR-REG-0A.G2
- new net PROG/BUS-SW: ADDR-R/P-SW-0A.!A!/B, ADDR-R/P-SW-1A.!A!/B, ADDR-R/P-SW-2A.!A!/B, ADDR-R/P-SW-3A.!A!/B, DATA-R/P-SW-0A.!A!/B, DATA-R/P-SW-1A.!A!/B, SW2.1
- net ADDR-A0: now also ADDR-R/P-SW-0A.1Y, BUFFER-0A.A5, LED2.A; no longer MEMORY-0-8KX8-6264.A0, MEMORY-1-8KX8-6264.A0, MEMORY-2-8KX8-6264.A0, MEMORY-3-8KX8-6264.A0
- net ADDR-A1: now also ADDR-R/P-SW-0A.2Y, BUFFER-0A.A6, LED3.A; no longer MEMORY-0-8KX8-6264.A1, MEMORY-1-8KX8-6264.A1, MEMORY-2-8KX8-6264.A1, MEMORY-3-8KX8-6264.A1
- net ADDR-A10: now also ADDR-R/P-SW-2A.3Y, BUFFER-1A.A7, LED16.A; no longer DEMUX-2X4-0A.A
- net ADDR-A11: now also ADDR-R/P-SW-2A.4Y, BUFFER-1A.A8, LED17.A; no longer DEMUX-2X4-0A.B
- net ADDR-A2: now also ADDR-R/P-SW-0A.3Y, BUFFER-0A.A7, LED4.A; no longer MEMORY-0-8KX8-6264.A2, MEMORY-1-8KX8-6264.A2, MEMORY-2-8KX8-6264.A2, MEMORY-3-8KX8-6264.A2
- net ADDR-A3: now also ADDR-R/P-SW-0A.4Y, BUFFER-0A.A8, LED5.A; no longer MEMORY-0-8KX8-6264.A3, MEMORY-1-8KX8-6264.A3, MEMORY-2-8KX8-6264.A3, MEMORY-3-8KX8-6264.A3
- net ADDR-A4: now also ADDR-R/P-SW-1A.1Y, BUFFER-1A.A1, LED6.A; no longer MEMORY-0-8KX8-6264.A4, MEMORY-1-8KX8-6264.A4, MEMORY-2-8KX8-6264.A4, MEMORY-3-8KX8-6264.A4
- net ADDR-A5: now also ADDR-R/P-SW-1A.2Y, BUFFER-1A.A2, LED7.A; no longer MEMORY-0-8KX8-6264.A5, MEMORY-1-8KX8-6264.A5, MEMORY-2-8KX8-6264.A5, MEMORY-3-8KX8-6264.A5
- net ADDR-A6: now also ADDR-R/P-SW-1A.3Y, BUFFER-1A.A3, LED11.A; no longer MEMORY-0-8KX8-6264.A6, MEMORY-1-8KX8-6264.A6, MEMORY-2-8KX8-6264.A6, MEMORY-3-8KX8-6264.A6
- net ADDR-A7: now also ADDR-R/P-SW-1A.4Y, BUFFER-1A.A4, LED8.A; no longer MEMORY-0-8KX8-6264.A7, MEMORY-1-8KX8-6264.A7, MEMORY-2-8KX8-6264.A7, MEMORY-2-8KX8-6264.A8, MEMORY-3-8KX8-6264.A7
- net ADDR-A8: now also ADDR-R/P-SW-2A.1Y, BUFFER-1A.A5, LED9.A; no longer MEMORY-0-8KX8-6264.A8, MEMORY-1-8KX8-6264.A8, MEMORY-3-8KX8-6264.A8
- net ADDR-A9: now also ADDR-R/P-SW-2A.2Y, BUFFER-1A.A6, LED10.A; no longer MEMORY-0-8KX8-6264.A9, MEMORY-1-8KX8-6264.A9, MEMORY-2-8KX8-6264.A9, MEMORY-3-8KX8-6264.A9
- net ADDR-B10: now also BUFFER-1A.B7; no longer PAGE-ADD-REG-1A.Q1, PAGE-ADDR-REG-0A.Q1, PAGE-ADDR-REG-2A.Q1, PAGE-ADDR-REG-3A.Q1
- net ADDR-B11: now also BUFFER-1A.B8; no longer PAGE-ADD-REG-1A.Q2, PAGE-ADDR-REG-0A.Q2, PAGE-ADDR-REG-2A.Q2, PAGE-ADDR-REG-3A.Q2
- net ADDR-B12: now also BUFFER-3A.B1; no longer PAGE-ADD-REG-1A.Q3, PAGE-ADDR-REG-0A.Q3, PAGE-ADDR-REG-2A.Q3, PAGE-ADDR-REG-3A.Q3
- net CLK-SIG: now also IC13A.CLK, IC14A.CLK, IC15A.CLK, IC16A.CLK; no longer PAGE-ADD-REG-1A.CLK, PAGE-ADDR-REG-2A.CLK, PAGE-ADDR-REG-3A.CLK
- net GND: now also ADDR-R/P-SW-0A.G, ADDR-R/P-SW-1A.G, ADDR-R/P-SW-2A.G, ADDR-R/P-SW-3A.2A, ADDR-R/P-SW-3A.2B, ADDR-R/P-SW-3A.2Y, ADDR-R/P-SW-3A.3A, ADDR-R/P-SW-3A.3B, ADDR-R/P-SW-3A.3Y, ADDR-R/P-SW-3A.4A, ADDR-R/P-SW-3A.4B, ADDR-R/P-SW-3A.4Y, ADDR-R/P-SW-3A.G, BUFFER-0A.G, BUFFER-1A.G, BUFFER-3A.A2, BUFFER-3A.A3, BUFFER-3A.A4, BUFFER-3A.A5, BUFFER-3A.A6, BUFFER-3A.A7, BUFFER-3A.A8, BUFFER-3A.B2, BUFFER-3A.B3, BUFFER-3A.B4, BUFFER-3A.B5, BUFFER-3A.B6, BUFFER-3A.B7, BUFFER-3A.B8, BUFFER-3A.G, C3.2, C4.1, DATA-R/P-SW-0A.G, DATA-R/P-SW-1A.G, IC10A.!CE, IC10A.!OE, IC11.GND, IC12A.G, IC16A.B, IC16A.C, IC16A.D, IC16A.QC, IC16A.QD, IC16A.RCO, IC18A.A6, IC18A.A7, IC18A.A8, IC18A.B6, IC18A.B7, IC18A.B8, IC9A.!Q, IC9B.!Q, IC9B.K, LED10.C, LED11.C, LED12.C, LED13.C, LED14.C, LED15.C, LED16.C, LED17.C, LED18.C, LED19.C, LED2.C, LED20.C, LED21.C, LED22.C, LED23.C, LED24.C, LED25.C, LED26.C, LED3.C, LED4.C, LED5.C, LED6.C, LED7.C, LED8.C, LED9.C, PROG/RUN-ADDR-SW.13, PROG/RUN-ADDR-SW.14, PROG/RUN-ADDR-SW.15, PROG/RUN-ADDR-SW.16, PROG/RUN-ADDR-SW.17, PROG/RUN-ADDR-SW.18, PROG/RUN-ADDR-SW.19, PROG/RUN-ADDR-SW.20, PROG/RUN-ADDR-SW.21, PROG/RUN-ADDR-SW.22, PROG/RUN-ADDR-SW.23, PROG/RUN-ADDR-SW.24, PROG/RUN-DATA-SW.10, PROG/RUN-DATA-SW.11, PROG/RUN-DATA-SW.12, PROG/RUN-DATA-SW.13, PROG/RUN-DATA-SW.14, PROG/RUN-DATA-SW.15, PROG/RUN-DATA-SW.16, PROG/RUN-DATA-SW.9, SW2.2, SW3.2; no longer MEMORY-0-8KX8-6264.NC, MEMORY-1-8KX8-6264.NC, MEMORY-2-8KX8-6264.NC, MEMORY-3-8KX8-6264.NC, PAGE-ADD-REG-1A.CLR, PAGE-ADD-REG-1A.M, PAGE-ADD-REG-1A.N, PAGE-ADD-REG-1A.Q4, PAGE-ADDR-REG-0A.Q4, PAGE-ADDR-REG-2A.CLR, PAGE-ADDR-REG-2A.M, PAGE-ADDR-REG-2A.N, PAGE-ADDR-REG-2A.Q4, PAGE-ADDR-REG-3A.CLR, PAGE-ADDR-REG-3A.M, PAGE-ADDR-REG-3A.N, PAGE-ADDR-REG-3A.Q4
- net MRQ: now also BUFFER-2A.G
- net VCC: now also BUFFER-0A.DIR, BUFFER-1A.DIR, BUFFER-3A.DIR, IC10A.!WE, IC11.R, IC11.V+, IC17A.DIR, IC18A.DIR, IC9A.CLR, IC9A.J, IC9A.K, IC9A.PRE, IC9B.CLR, IC9B.J, IC9B.PRE, R9.1
- net WR: now also BUFFER-2A.DIR
Other:
- note added: "Numerical Display"
- note added: "PROGRAM COUNTER"
- note added: "SRAM (STATIC RANDOM ACCESS MEMORY) 4x8K"
- note removed: "SRAM (STATIC RANDOM MEMORY ACCESS) 4x8K"
- moved on the sheet: 4BIT-FULL-ADDER-2, 4BIT-FULL-ADDER-3, C1, C2, CLK, DEMUX-2X4-0A, DUAL-4X1-MUX-0, DUAL-4X1-MUX-1, DUAL-4X1-MUX-2, DUAL-4X1-MUX-3, IC1A, IC2A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

Commit message: Added General Purpose Registers to the 8bit computer schema
Parts:
- added LED0, LED27, LED28, LED29, LED30, LED31, LED32, LED33, LED34, LED35, LED36, LED37, LED38, LED39, LED40, LED41, LED42, LED43, LED44, LED45, LED46, LED47, LED48, LED49, LED50, LED51, LED52, LED53, LED54, LED55, LED56, LED57, LED58, LED59, LED60, LED61, LED62, LED63, LED64, LED65, LED66, LED67, LED68, LED69, LED70, LED71, LED72, LED73, LED74, LED75, LED76, LED77, LED78, LED79, LED80, LED81, LED82, LED83, LED84, LED85, LED86, LED87, LED88, LED89: (no value), led:LED5MM
- added REG-AC-BUF, REG-IO0-BUF, REG-IO1-BUF, REG-IO2-BUF, REG-IO3-BUF, REG-IR-BUF, REG-MAR-BUF, REG-MBR-BUF: 74LS245N, 74xx-eu:74LS245N
- added REG-AC-H, REG-AC-L, REG-IO0-H, REG-IO0-L, REG-IO1-H, REG-IO1-L, REG-IO2-H, REG-IO2-L, REG-IO3-H, REG-IO3-L, REG-IR-H, REG-IR-L, REG-MAR-H, REG-MAR-L, REG-MBR-H, REG-MBR-L: 74LS173N, 74xx-eu:74LS173N
Connections:
- new net DATA-IR0: REG-IR-BUFA.B5
- new net DATA-IR1: REG-IR-BUFA.B6
- new net DATA-IR2: REG-IR-BUFA.B7
- new net DATA-IR3: REG-IR-BUFA.B8
- new net REG-AC-DATA0: LED0.A, REG-AC-BUFA.A1, REG-AC-LA.Q1
- new net REG-AC-DATA1: LED33.A, REG-AC-BUFA.A2, REG-AC-LA.Q2
- new net REG-AC-DATA2: LED32.A, REG-AC-BUFA.A3, REG-AC-LA.Q3
- new net REG-AC-DATA3: LED31.A, REG-AC-BUFA.A4, REG-AC-LA.Q4
- new net REG-AC-DATA4: LED30.A, REG-AC-BUFA.A5, REG-AC-HA.Q1
- new net REG-AC-DATA5: LED29.A, REG-AC-BUFA.A6, REG-AC-HA.Q2
- new net REG-AC-DATA6: LED28.A, REG-AC-BUFA.A7, REG-AC-HA.Q3
- new net REG-AC-DATA7: LED27.A, REG-AC-BUFA.A8, REG-AC-HA.Q4
- new net REG-ACU-LOAD-IN: REG-AC-HA.G1, REG-AC-HA.G2, REG-AC-LA.G1, REG-AC-LA.G2
- new net REG-IO0-DATA0: LED58.A, REG-IO0-BUFA.A1, REG-IO0-LA.Q1
- new net REG-IO0-DATA1: LED59.A, REG-IO0-BUFA.A2, REG-IO0-LA.Q2
- new net REG-IO0-DATA2: LED60.A, REG-IO0-BUFA.A3, REG-IO0-LA.Q3
- new net REG-IO0-DATA3: LED61.A, REG-IO0-BUFA.A4, REG-IO0-LA.Q4
- new net REG-IO0-DATA4: LED62.A, REG-IO0-BUFA.A5, REG-IO0-HA.Q1
- new net REG-IO0-DATA5: LED63.A, REG-IO0-BUFA.A6, REG-IO0-HA.Q2
- new net REG-IO0-DATA6: LED64.A, REG-IO0-BUFA.A7, REG-IO0-HA.Q3
- new net REG-IO0-DATA7: LED65.A, REG-IO0-BUFA.A8, REG-IO0-HA.Q4
- new net REG-IO0-LOAD-IN: REG-IO0-HA.G1, REG-IO0-HA.G2, REG-IO0-LA.G1, REG-IO0-LA.G2
- new net REG-IO0-LOAD-OUT: REG-IO0-BUFA.G
- new net REG-IO1-DATA0: LED66.A, REG-IO1-BUFA.A1, REG-IO1-LA.Q1
- new net REG-IO1-DATA1: LED67.A, REG-IO1-BUFA.A2, REG-IO1-LA.Q2
- new net REG-IO1-DATA2: LED68.A, REG-IO1-BUFA.A3, REG-IO1-LA.Q3
- new net REG-IO1-DATA3: LED69.A, REG-IO1-BUFA.A4, REG-IO1-LA.Q4
- new net REG-IO1-DATA4: LED70.A, REG-IO1-BUFA.A5, REG-IO1-HA.Q1
- new net REG-IO1-DATA5: LED71.A, REG-IO1-BUFA.A6, REG-IO1-HA.Q2
- new net REG-IO1-DATA6: LED72.A, REG-IO1-BUFA.A7, REG-IO1-HA.Q3
- new net REG-IO1-DATA7: LED73.A, REG-IO1-BUFA.A8, REG-IO1-HA.Q4
- new net REG-IO1-LOAD-IN: REG-IO1-HA.G1, REG-IO1-HA.G2, REG-IO1-LA.G1, REG-IO1-LA.G2
- new net REG-IO1-LOAD-OUT: REG-IO1-BUFA.G
- new net REG-IO2-DATA0: LED74.A, REG-IO2-BUFA.A1, REG-IO2-LA.Q1
- new net REG-IO2-DATA1: LED75.A, REG-IO2-BUFA.A2, REG-IO2-LA.Q2
- new net REG-IO2-DATA2: LED76.A, REG-IO2-BUFA.A3, REG-IO2-LA.Q3
- new net REG-IO2-DATA3: LED77.A, REG-IO2-BUFA.A4, REG-IO2-LA.Q4
- new net REG-IO2-DATA4: LED78.A, REG-IO2-BUFA.A5, REG-IO2-HA.Q1
- new net REG-IO2-DATA5: LED79.A, REG-IO2-BUFA.A6, REG-IO2-HA.Q2
- new net REG-IO2-DATA6: LED80.A, REG-IO2-BUFA.A7, REG-IO2-HA.Q3
- new net REG-IO2-DATA7: LED81.A, REG-IO2-BUFA.A8, REG-IO2-HA.Q4
- new net REG-IO2-LOAD-IN: REG-IO2-HA.G1, REG-IO2-HA.G2, REG-IO2-LA.G1, REG-IO2-LA.G2
- new net REG-IO2-LOAD-OUT: REG-IO2-BUFA.G
- new net REG-IO3-DATA0: LED82.A, REG-IO3-BUFA.A1, REG-IO3-LA.Q1
- new net REG-IO3-DATA1: LED83.A, REG-IO3-BUFA.A2, REG-IO3-LA.Q2
- new net REG-IO3-DATA2: LED84.A, REG-IO3-BUFA.A3, REG-IO3-LA.Q3
- new net REG-IO3-DATA3: LED85.A, REG-IO3-BUFA.A4, REG-IO3-LA.Q4
- new net REG-IO3-DATA4: LED86.A, REG-IO3-BUFA.A5, REG-IO3-HA.Q1
- new net REG-IO3-DATA5: LED87.A, REG-IO3-BUFA.A6, REG-IO3-HA.Q2
- new net REG-IO3-DATA6: LED88.A, REG-IO3-BUFA.A7, REG-IO3-HA.Q3
- new net REG-IO3-DATA7: LED89.A, REG-IO3-BUFA.A8, REG-IO3-HA.Q4
- new net REG-IO3-LOAD-IN: REG-IO3-HA.G1, REG-IO3-HA.G2, REG-IO3-LA.G1, REG-IO3-LA.G2
- new net REG-IO3-LOAD-OUT: REG-IO3-BUFA.G
- new net REG-IR-DATA0: LED50.A, REG-IR-BUFA.A1, REG-IR-LA.Q1
- new net REG-IR-DATA1: LED51.A, REG-IR-BUFA.A2, REG-IR-LA.Q2
- new net REG-IR-DATA2: LED52.A, REG-IR-BUFA.A3, REG-IR-LA.Q3
- new net REG-IR-DATA3: LED53.A, REG-IR-BUFA.A4, REG-IR-LA.Q4
- new net REG-IR-DATA4: LED54.A, REG-IR-BUFA.A5, REG-IR-HA.Q1
- new net REG-IR-DATA5: LED55.A, REG-IR-BUFA.A6, REG-IR-HA.Q2
- new net REG-IR-DATA6: LED56.A, REG-IR-BUFA.A7, REG-IR-HA.Q3
- new net REG-IR-DATA7: LED57.A, REG-IR-BUFA.A8, REG-IR-HA.Q4
- new net REG-IR-LOAD-IN: REG-IR-HA.G1, REG-IR-HA.G2, REG-IR-LA.G1, REG-IR-LA.G2
- new net REG-IR-LOAD-OUT: REG-IR-BUFA.G
- new net REG-MAR-DATA0: LED42.A, REG-MAR-BUFA.A1, REG-MAR-LA.Q1
- new net REG-MAR-DATA1: LED43.A, REG-MAR-BUFA.A2, REG-MAR-LA.Q2
- new net REG-MAR-DATA2: LED44.A, REG-MAR-BUFA.A3, REG-MAR-LA.Q3
- new net REG-MAR-DATA3: LED45.A, REG-MAR-BUFA.A4, REG-MAR-LA.Q4
- new net REG-MAR-DATA4: LED46.A, REG-MAR-BUFA.A5, REG-MAR-HA.Q1
- new net REG-MAR-DATA5: LED47.A, REG-MAR-BUFA.A6, REG-MAR-HA.Q2
- new net REG-MAR-DATA6: LED48.A, REG-MAR-BUFA.A7, REG-MAR-HA.Q3
- new net REG-MAR-DATA7: LED49.A, REG-MAR-BUFA.A8, REG-MAR-HA.Q4
- new net REG-MAR-LOAD-IN: REG-MAR-HA.G1, REG-MAR-HA.G2, REG-MAR-LA.G1, REG-MAR-LA.G2
- new net REG-MAR-LOAD-OUT: REG-MAR-BUFA.G
- new net REG-MBR-DATA0: LED34.A, REG-MBR-BUFA.A1, REG-MBR-LA.Q1
- new net REG-MBR-DATA1: LED35.A, REG-MBR-BUFA.A2, REG-MBR-LA.Q2
- new net REG-MBR-DATA2: LED36.A, REG-MBR-BUFA.A3, REG-MBR-LA.Q3
- new net REG-MBR-DATA3: LED37.A, REG-MBR-BUFA.A4, REG-MBR-LA.Q4
- new net REG-MBR-DATA4: LED38.A, REG-MBR-BUFA.A5, REG-MBR-HA.Q1
- new net REG-MBR-DATA5: LED39.A, REG-MBR-BUFA.A6, REG-MBR-HA.Q2
- new net REG-MBR-DATA6: LED40.A, REG-MBR-BUFA.A7, REG-MBR-HA.Q3
- new net REG-MBR-DATA7: LED41.A, REG-MBR-BUFA.A8, REG-MBR-HA.Q4
- new net REG-MBR-LOAD-IN: REG-MBR-HA.G1, REG-MBR-HA.G2, REG-MBR-LA.G1, REG-MBR-LA.G2
- new net REG-MBR-LOAD-OUT: REG-MBR-BUFA.G
- new net REG-SC-LOAD-OUT: REG-AC-BUFA.G
- net CLK-SIG: now also REG-AC-HA.CLK, REG-AC-LA.CLK, REG-IO0-HA.CLK, REG-IO0-LA.CLK, REG-IO1-HA.CLK, REG-IO1-LA.CLK, REG-IO2-HA.CLK, REG-IO2-LA.CLK, REG-IO3-HA.CLK, REG-IO3-LA.CLK, REG-IR-HA.CLK, REG-IR-LA.CLK, REG-MAR-HA.CLK, REG-MAR-LA.CLK, REG-MBR-HA.CLK, REG-MBR-LA.CLK
- net DATA-BUS0: now also REG-AC-BUFA.B1, REG-AC-LA.D1, REG-IO0-BUFA.B1, REG-IO0-LA.D1, REG-IO1-BUFA.B1, REG-IO1-LA.D1, REG-IO2-BUFA.B1, REG-IO2-LA.D1, REG-IO3-BUFA.B1, REG-IO3-LA.D1, REG-IR-BUFA.B1, REG-IR-LA.D1, REG-MAR-BUFA.B1, REG-MAR-LA.D1, REG-MBR-BUFA.B1, REG-MBR-LA.D1
- net DATA-BUS1: now also REG-AC-BUFA.B2, REG-AC-LA.D2, REG-IO0-BUFA.B2, REG-IO0-LA.D2, REG-IO1-BUFA.B2, REG-IO1-LA.D2, REG-IO2-BUFA.B2, REG-IO2-LA.D2, REG-IO3-BUFA.B2, REG-IO3-LA.D2, REG-IR-BUFA.B2, REG-IR-LA.D2, REG-MAR-BUFA.B2, REG-MAR-LA.D2, REG-MBR-BUFA.B2, REG-MBR-LA.D2
- net DATA-BUS2: now also REG-AC-BUFA.B3, REG-AC-LA.D3, REG-IO0-BUFA.B3, REG-IO0-LA.D3, REG-IO1-BUFA.B3, REG-IO1-LA.D3, REG-IO2-BUFA.B3, REG-IO2-LA.D3, REG-IO3-BUFA.B3, REG-IO3-LA.D3, REG-IR-BUFA.B3, REG-IR-LA.D3, REG-MAR-BUFA.B3, REG-MAR-LA.D3, REG-MBR-BUFA.B3, REG-MBR-LA.D3
- net DATA-BUS3: now also REG-AC-BUFA.B4, REG-AC-LA.D4, REG-IO0-BUFA.B4, REG-IO0-LA.D4, REG-IO1-BUFA.B4, REG-IO1-LA.D4, REG-IO2-BUFA.B4, REG-IO2-LA.D4, REG-IO3-BUFA.B4, REG-IO3-LA.D4, REG-IR-BUFA.B4, REG-IR-LA.D4, REG-MAR-BUFA.B4, REG-MAR-LA.D4, REG-MBR-BUFA.B4, REG-MBR-LA.D4
- net DATA-BUS4: now also REG-AC-BUFA.B5, REG-AC-HA.D1, REG-IO0-BUFA.B5, REG-IO0-HA.D1, REG-IO1-BUFA.B5, REG-IO1-HA.D1, REG-IO2-BUFA.B5, REG-IO2-HA.D1, REG-IO3-BUFA.B5, REG-IO3-HA.D1, REG-IR-HA.D1, REG-MAR-BUFA.B5, REG-MAR-HA.D1, REG-MBR-BUFA.B5, REG-MBR-HA.D1
- net DATA-BUS5: now also REG-AC-BUFA.B6, REG-AC-HA.D2, REG-IO0-BUFA.B6, REG-IO0-HA.D2, REG-IO1-BUFA.B6, REG-IO1-HA.D2, REG-IO2-BUFA.B6, REG-IO2-HA.D2, REG-IO3-BUFA.B6, REG-IO3-HA.D2, REG-IR-HA.D2, REG-MAR-BUFA.B6, REG-MAR-HA.D2, REG-MBR-BUFA.B6, REG-MBR-HA.D2
- net DATA-BUS6: now also REG-AC-BUFA.B7, REG-AC-HA.D3, REG-IO0-BUFA.B7, REG-IO0-HA.D3, REG-IO1-BUFA.B7, REG-IO1-HA.D3, REG-IO2-BUFA.B7, REG-IO2-HA.D3, REG-IO3-BUFA.B7, REG-IO3-HA.D3, REG-IR-HA.D3, REG-MAR-BUFA.B7, REG-MAR-HA.D3, REG-MBR-BUFA.B7, REG-MBR-HA.D3
- net DATA-BUS7: now also REG-AC-BUFA.B8, REG-AC-HA.D4, REG-IO0-BUFA.B8, REG-IO0-HA.D4, REG-IO1-BUFA.B8, REG-IO1-HA.D4, REG-IO2-BUFA.B8, REG-IO2-HA.D4, REG-IO3-BUFA.B8, REG-IO3-HA.D4, REG-IR-HA.D4, REG-MAR-BUFA.B8, REG-MAR-HA.D4, REG-MBR-BUFA.B8, REG-MBR-HA.D4
- net GND: now also LED0.C, LED27.C, LED28.C, LED29.C, LED30.C, LED31.C, LED32.C, LED33.C, LED34.C, LED35.C, LED36.C, LED37.C, LED38.C, LED39.C, LED40.C, LED41.C, LED42.C, LED43.C, LED44.C, LED45.C, LED46.C, LED47.C, LED48.C, LED49.C, LED50.C, LED51.C, LED52.C, LED53.C, LED54.C, LED55.C, LED56.C, LED57.C, LED58.C, LED59.C, LED60.C, LED61.C, LED62.C, LED63.C, LED64.C, LED65.C, LED66.C, LED67.C, LED68.C, LED69.C, LED70.C, LED71.C, LED72.C, LED73.C, LED74.C, LED75.C, LED76.C, LED77.C, LED78.C, LED79.C, LED80.C, LED81.C, LED82.C, LED83.C, LED84.C, LED85.C, LED86.C, LED87.C, LED88.C, LED89.C, REG-AC-HA.CLR, REG-AC-HA.M, REG-AC-HA.N, REG-AC-LA.CLR, REG-AC-LA.M, REG-AC-LA.N, REG-IO0-HA.CLR, REG-IO0-HA.M, REG-IO0-HA.N, REG-IO0-LA.CLR, REG-IO0-LA.M, REG-IO0-LA.N, REG-IO1-HA.CLR, REG-IO1-HA.M, REG-IO1-HA.N, REG-IO1-LA.CLR, REG-IO1-LA.M, REG-IO1-LA.N, REG-IO2-HA.CLR, REG-IO2-HA.M, REG-IO2-HA.N, REG-IO2-LA.CLR, REG-IO2-LA.M, REG-IO2-LA.N, REG-IO3-HA.CLR, REG-IO3-HA.M, REG-IO3-HA.N, REG-IO3-LA.CLR, REG-IO3-LA.M, REG-IO3-LA.N, REG-IR-HA.CLR, REG-IR-HA.M, REG-IR-HA.N, REG-IR-LA.CLR, REG-IR-LA.M, REG-IR-LA.N, REG-MAR-HA.CLR, REG-MAR-HA.M, REG-MAR-HA.N, REG-MAR-LA.CLR, REG-MAR-LA.M, REG-MAR-LA.N, REG-MBR-HA.CLR, REG-MBR-HA.M, REG-MBR-HA.N, REG-MBR-LA.CLR, REG-MBR-LA.M, REG-MBR-LA.N
- net VCC: now also REG-AC-BUFA.DIR, REG-IO0-BUFA.DIR, REG-IO1-BUFA.DIR, REG-IO2-BUFA.DIR, REG-IO3-BUFA.DIR, REG-IR-BUFA.DIR, REG-MAR-BUFA.DIR, REG-MBR-BUFA.DIR
Other:
- note added: "General Purpose Registers"
- moved on the sheet: ADDR-R/P-SW-0, ADDR-R/P-SW-1, ADDR-R/P-SW-2, ADDR-R/P-SW-3, BUFFER-0, BUFFER-1, BUFFER-2, BUFFER-3, C3, C4, D1, D2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

Commit message: Connected IPs to the mainband on general schema
Parts:
- removed R4: 2.2k, resistor:R-EU_0204/5
- LED1: device eagle-ltspice:LED_ELD260 -> led:LED5MM
- renumbered REG-AC-H to REG-ACU-H, REG-AC-L to REG-ACU-L
Connections:
- removed net ALU-A0-IN: IC1A.I, IC35D.I1, IC37D.I0, IC46A.I1
- removed net ALU-A1-IN: IC2A.I, IC38A.I0, IC39A.I1, IC46B.I1
- removed net ALU-A2-IN: IC3A.I, IC41D.I0, IC42D.I1, IC46C.I1
- removed net ALU-A3-IN: IC44A.I0, IC45A.I1, IC46D.I1, IC4A.I
- removed net ALU-A4-IN: IC47A.I1, IC48D.I1, IC50D.I0, IC5A.I
- removed net ALU-A5-IN: IC47B.I1, IC51A.I0, IC52A.I1, IC6A.I
- removed net ALU-A6-IN: IC47C.I1, IC54D.I0, IC55D.I1, IC7A.I
- removed net ALU-A7-IN: IC47D.I1, IC57A.I0, IC58A.I1, IC8A.I
- removed net ALU-B0-IN: 4BIT-FULL-ADDER-2A.B1, IC35D.I0, IC37D.I1
- removed net ALU-B1-IN: 4BIT-FULL-ADDER-2A.B2, IC38A.I1, IC39A.I0
- removed net ALU-B2-IN: 4BIT-FULL-ADDER-2A.B3, IC41D.I1, IC42D.I0
- removed net ALU-B3-IN: 4BIT-FULL-ADDER-2A.B4, IC44A.I1, IC45A.I0
- removed net ALU-B4-IN: 4BIT-FULL-ADDER-3A.B1, IC48D.I0, IC50D.I1
- removed net ALU-B5-IN: 4BIT-FULL-ADDER-3A.B2, IC51A.I1, IC52A.I0
- removed net ALU-B6-IN: 4BIT-FULL-ADDER-3A.B3, IC54D.I1, IC55D.I0
- removed net ALU-B7-IN: 4BIT-FULL-ADDER-3A.B4, IC57A.I1, IC58A.I0
- removed net ALU-C0-BUS-IN: IC59A.B1
- removed net ALU-C1-BUS-IN: IC59A.B2
- removed net ALU-C2-BUS-IN: IC59A.B3
- removed net ALU-C3-BUS-IN: IC59A.B4
- removed net ALU-C4-BUS-IN: IC59A.B5
- removed net ALU-C5-BUS-IN: IC59A.B6
- removed net ALU-C6-BUS-IN: IC59A.B7
- removed net ALU-C7-BUS-IN: IC59A.B8
- removed net DATA-A0: BUFFER-2A.B1, DATA-R/P-SW-0A.1Y, IC18A.B2, PAGE-ADDR-REG-0A.D1
- removed net DATA-A1: BUFFER-2A.B2, DATA-R/P-SW-0A.2Y, IC18A.B3, PAGE-ADDR-REG-0A.D2
- removed net DATA-A2: BUFFER-2A.B3, DATA-R/P-SW-0A.3Y, IC18A.B4, PAGE-ADDR-REG-0A.D3
- removed net DATA-A3: BUFFER-2A.B4, DATA-R/P-SW-0A.4Y, IC18A.B5, PAGE-ADDR-REG-0A.D4
- removed net DATA-A4: BUFFER-2A.B5, DATA-R/P-SW-1A.1Y
- removed net DATA-A5: BUFFER-2A.B6, DATA-R/P-SW-1A.2Y
- removed net DATA-A6: BUFFER-2A.B7, DATA-R/P-SW-1A.3Y
- removed net DATA-A7: BUFFER-2A.B8, DATA-R/P-SW-1A.4Y
- removed net DATA-BUS8: IC18A.B1
- removed net N$4: LED1.C, R4.1
- removed net REG-AC-DATA0: LED0.A, REG-AC-BUFA.A1, REG-ACU-LA.Q1
- removed net REG-AC-DATA1: LED33.A, REG-AC-BUFA.A2, REG-ACU-LA.Q2
- removed net REG-AC-DATA2: LED32.A, REG-AC-BUFA.A3, REG-ACU-LA.Q3
- removed net REG-AC-DATA3: LED31.A, REG-AC-BUFA.A4, REG-ACU-LA.Q4
- removed net REG-AC-DATA5: LED29.A, REG-AC-BUFA.A6, REG-ACU-HA.Q2
- removed net REG-AC-DATA6: LED28.A, REG-AC-BUFA.A7, REG-ACU-HA.Q3
- new net REG-ACU-DATA0: IC1A.I, IC35D.I1, IC37D.I0, IC46A.I1, LED0.A, REG-AC-BUFA.A1, REG-ACU-LA.Q1
- new net REG-ACU-DATA1: IC2A.I, IC38A.I0, IC39A.I1, IC46B.I1, LED33.A, REG-AC-BUFA.A2, REG-ACU-LA.Q2
- new net REG-ACU-DATA2: IC3A.I, IC41D.I0, IC42D.I1, IC46C.I1, LED32.A, REG-AC-BUFA.A3, REG-ACU-LA.Q3
- new net REG-ACU-DATA3: IC44A.I0, IC45A.I1, IC46D.I1, IC4A.I, LED31.A, REG-AC-BUFA.A4, REG-ACU-LA.Q4
- new net REG-ACU-DATA4: IC47A.I1, IC48D.I1, IC50D.I0, IC5A.I, REG-ACU-HA.Q1
- new net REG-ACU-DATA5: IC47B.I1, IC51A.I0, IC52A.I1, IC6A.I, LED29.A, REG-AC-BUFA.A6, REG-ACU-HA.Q2
- new net REG-ACU-DATA6: IC47C.I1, IC54D.I0, IC55D.I1, IC7A.I, LED28.A, REG-AC-BUFA.A7, REG-ACU-HA.Q3
- new net REG-ACU-DATA7: IC47D.I1, IC57A.I0, IC58A.I1, IC8A.I, REG-ACU-HA.Q4
- net ADDR-BUS0: now also IC17A.B1
- net ADDR-BUS1: now also IC17A.B2
- net ADDR-BUS2: now also IC17A.B3
- net ADDR-BUS3: now also IC17A.B4
- net ADDR-BUS4: now also IC17A.B5
- net ADDR-BUS5: now also IC17A.B6
- net ADDR-BUS6: now also IC17A.B7
- net ADDR-BUS7: now also IC17A.B8
- net ADDR-BUS8: now also IC18A.B1
- net ADDR-PAGE10: now also IC18A.B3
- net ADDR-PAGE11: now also IC18A.B4
- net ADDR-PAGE12: now also IC18A.B5
- net ADDR-PAGE9: now also IC18A.B2
- net CLK-SIG: now also LED1.C
- net DATA-BUS0: now also BUFFER-2A.B1, DATA-R/P-SW-0A.1Y, IC59A.B1, PAGE-ADDR-REG-0A.D1; no longer IC17A.B1
- net DATA-BUS1: now also BUFFER-2A.B2, DATA-R/P-SW-0A.2Y, IC59A.B2, PAGE-ADDR-REG-0A.D2; no longer IC17A.B2
- net DATA-BUS2: now also BUFFER-2A.B3, DATA-R/P-SW-0A.3Y, IC59A.B3, PAGE-ADDR-REG-0A.D3; no longer IC17A.B3
- net DATA-BUS3: now also BUFFER-2A.B4, DATA-R/P-SW-0A.4Y, IC59A.B4, PAGE-ADDR-REG-0A.D4; no longer IC17A.B4
- net DATA-BUS4: now also BUFFER-2A.B5, DATA-R/P-SW-1A.1Y, IC59A.B5; no longer IC17A.B5
- net DATA-BUS5: now also BUFFER-2A.B6, DATA-R/P-SW-1A.2Y, IC59A.B6; no longer IC17A.B6
- net DATA-BUS6: now also BUFFER-2A.B7, DATA-R/P-SW-1A.3Y, IC59A.B7; no longer IC17A.B7
- net DATA-BUS7: now also BUFFER-2A.B8, DATA-R/P-SW-1A.4Y, IC59A.B8; no longer IC17A.B8
- net GND: no longer R4.2
- net REG-AC-DATA4: no longer REG-ACU-HA.Q1
- net REG-AC-DATA7: no longer REG-ACU-HA.Q4
- net REG-MBR-DATA0: now also 4BIT-FULL-ADDER-2A.B1, IC35D.I0, IC37D.I1
- net REG-MBR-DATA1: now also 4BIT-FULL-ADDER-2A.B2, IC38A.I1, IC39A.I0
- net REG-MBR-DATA2: now also 4BIT-FULL-ADDER-2A.B3, IC41D.I1, IC42D.I0
- net REG-MBR-DATA3: now also 4BIT-FULL-ADDER-2A.B4, IC44A.I1, IC45A.I0
- net REG-MBR-DATA4: now also 4BIT-FULL-ADDER-3A.B1, IC48D.I0, IC50D.I1
- net REG-MBR-DATA5: now also 4BIT-FULL-ADDER-3A.B2, IC51A.I1, IC52A.I0
- net REG-MBR-DATA6: now also 4BIT-FULL-ADDER-3A.B3, IC54D.I1, IC55D.I0
- net REG-MBR-DATA7: now also 4BIT-FULL-ADDER-3A.B4, IC57A.I1, IC58A.I0
Other:
- note added: "GENERAL PURPOSE REGISTERS"
- note added: "NUMERICAL DISPLAY"
- note removed: "General Purpose Registers"
- note removed: "Numerical Display"
- moved on the sheet: BUFFER-2, DATA-R/P-SW-0, DATA-R/P-SW-1, IC13, IC14, IC15, IC16, IC17, IC18, IC19A, IC59, PAGE-ADDR-REG-0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

Commit message: Changed PC - SRAM connections, to enable ADDR load on DATA BUS
Parts:
- renumbered IC13 to PC0, IC14 to PC1, IC15 to PC2, IC16 to PC3
Connections:
- net PAGE-EN-A0 renamed MEM-EN-A0
- net PAGE-EN-A1 renamed MEM-EN-A1
- net PAGE-EN-A2 renamed MEM-EN-A2
- net PAGE-EN-A3 renamed MEM-EN-A3
- net PAGE-EN-B0 renamed MEM-EN-B0
- net PAGE-EN-B1 renamed MEM-EN-B1
- net PAGE-EN-B2 renamed MEM-EN-B2
- net PAGE-EN-B3 renamed MEM-EN-B3
- removed net COUNTER-OUT: IC17A.G, IC18A.G
- removed net DATA-OUT0: IC17A.A1, PC0A.QA
- removed net DATA-OUT1: IC17A.A2, PC0A.QB
- removed net DATA-OUT10: IC18A.A3, PC2A.QC
- removed net DATA-OUT11: IC18A.A4, PC2A.QD
- removed net DATA-OUT12: IC18A.A5, PC3A.QA
- removed net DATA-OUT2: IC17A.A3, PC0A.QC
- removed net DATA-OUT3: IC17A.A4, PC0A.QD
- removed net DATA-OUT4: IC17A.A5, PC1A.QA
- removed net DATA-OUT5: IC17A.A6, PC1A.QB
- removed net DATA-OUT6: IC17A.A7, PC1A.QC
- removed net DATA-OUT7: IC17A.A8, PC1A.QD
- removed net DATA-OUT8: IC18A.A1, PC2A.QA
- removed net DATA-OUT9: IC18A.A2, PC2A.QB
- new net ADDR-BUS11: ADDR-R/P-SW-2A.4A, IC18A.A4, PC2A.QD
- new net ADDR-BUS12: ADDR-R/P-SW-3A.1A, IC18A.A5, PC3A.QA
- new net COUNTER0-OUT: IC17A.G
- new net COUNTER1-OUT: IC18A.G
- net ADDR-BUS0: now also IC17A.A1, PC0A.QA; no longer IC17A.B1, PC0A.A
- net ADDR-BUS1: now also IC17A.A2, PC0A.QB; no longer IC17A.B2, PC0A.B
- net ADDR-BUS10: now also ADDR-R/P-SW-2A.3A, IC18A.A3, PC2A.QC; no longer DEMUX-2X4-0A.B
- net ADDR-BUS2: now also IC17A.A3, PC0A.QC; no longer IC17A.B3, PC0A.C
- net ADDR-BUS3: now also IC17A.A4, PC0A.QD; no longer IC17A.B4, PC0A.D
- net ADDR-BUS4: now also IC17A.A5, PC1A.QA; no longer IC17A.B5, PC1A.A
- net ADDR-BUS5: now also IC17A.A6, PC1A.QB; no longer IC17A.B6, PC1A.B
- net ADDR-BUS6: now also IC17A.A7, PC1A.QC; no longer IC17A.B7, PC1A.C
- net ADDR-BUS7: now also IC17A.A8, PC1A.QD; no longer IC17A.B8, PC1A.D
- net ADDR-BUS8: now also IC18A.A1, PC2A.QA; no longer IC18A.B1, PC2A.A
- net ADDR-BUS9: now also ADDR-R/P-SW-2A.2A, IC18A.A2, PC2A.QB; no longer DEMUX-2X4-0A.A
- net ADDR-PAGE10: no longer ADDR-R/P-SW-2A.3A, IC18A.B3
- net ADDR-PAGE11: no longer ADDR-R/P-SW-2A.4A, IC18A.B4
- net ADDR-PAGE12: no longer ADDR-R/P-SW-3A.1A, IC18A.B5
- net ADDR-PAGE9: no longer ADDR-R/P-SW-2A.2A, IC18A.B2
- net DATA-BUS0: now also IC17A.B1, IC18A.B1
- net DATA-BUS1: now also IC17A.B2, IC18A.B2
- net DATA-BUS2: now also IC17A.B3, IC18A.B3
- net DATA-BUS3: now also IC17A.B4, IC18A.B4
- net DATA-BUS4: now also IC17A.B5, IC18A.B5
- net DATA-BUS5: now also IC17A.B6, IC18A.B6
- net DATA-BUS6: now also IC17A.B7, IC18A.B7
- net DATA-BUS7: now also IC17A.B8, IC18A.B8
- net GND: no longer IC18A.B6, IC18A.B7, IC18A.B8
- net REG-IR-DATA0: now also PC2A.A
- net REG-IR-DATA1: now also DEMUX-2X4-0A.A
- net REG-IR-DATA2: now also DEMUX-2X4-0A.B
- net REG-MAR-DATA0: now also PC0A.A
- net REG-MAR-DATA1: now also PC0A.B
- net REG-MAR-DATA2: now also PC0A.C
- net REG-MAR-DATA3: now also PC0A.D
- net REG-MAR-DATA4: now also PC1A.A
- net REG-MAR-DATA5: now also PC1A.B
- net REG-MAR-DATA6: now also PC1A.C
- net REG-MAR-DATA7: now also PC1A.D

Commit message: Fixed chip names on main schema
Parts:
- renumbered BUFFER-0 to MEM-INT-BUF-0, BUFFER-1 to MEM-INT-BUF-1, BUFFER-2 to MEM-BUF, BUFFER-3 to MEM-INT-BUF-2, D1 to SEG-DISP0, D2 to SEG-DISP1, D3 to SEG-DISP2, D4 to SEG-DISP3, IC10 to EEPROM-AT28C16, IC11 to SEG-SWITCH, IC17 to PC-BUF-L, IC18 to PC-BUF-H, IC19 to RST-INVERTER, IC59 to ALU-BUF, IC9 to JK-FLIP-FLOP
