File: rel-8bit-computer.sch (EAGLE design)
At the start: 200 parts, among them IC1 74LS04N, IC12 74LS139N, IC2 74LS04N, IC3 74LS04N, IC35 74LS32N, IC37 74LS08N, IC38 74LS08N, IC39 74LS32N, IC4 74LS04N, IC41 74LS08N, IC42 74LS32N, IC44 74LS08N, IC45 74LS32N, IC46 74LS86N, IC47 74LS86N, IC48 74LS32N, IC5 74LS04N, IC50 74LS08N, IC51 74LS08N, IC52 74LS32N, IC54 74LS08N, IC55 74LS32N, IC57 74LS08N, IC58 74LS32N, IC6 74LS04N, IC7 74LS04N, IC8 74LS04N, Q1 BC556, Q2 BS170

Commit message: Added additional buffer to pull-up signals on diect connection to ALU
Parts:
- added REG-ACU-BUF1, REG-MBR-BUF1: 74LS245N, 74xx-eu:74LS245N
- renumbered REG-AC-BUF to REG-ACU-BUF0, REG-MBR-BUF to REG-MBR-BUF0
Connections:
- removed net ALU_EO: ALU-BUFA.G
- removed net REG-AC-DATA4: LED30.A, REG-ACU-BUF0A.A5
- removed net REG-AC-DATA7: LED27.A, REG-ACU-BUF0A.A8
- new net ACU-DATA0: IC1A.I, IC35D.I1, IC37D.I0, REG-ACU-BUF1A.B1
- new net ACU-DATA1: IC2A.I, IC38A.I0, IC39A.I1, REG-ACU-BUF1A.B2
- new net ACU-DATA2: IC3A.I, IC41D.I0, IC42D.I1, REG-ACU-BUF1A.B3
- new net ACU-DATA3: IC44A.I0, IC45A.I1, IC4A.I, REG-ACU-BUF1A.B4
- new net ACU-DATA4: IC48D.I1, IC50D.I0, IC5A.I, REG-ACU-BUF1A.B5
- new net ACU-DATA5: IC51A.I0, IC52A.I1, IC6A.I, REG-ACU-BUF1A.B6
- new net ACU-DATA6: IC54D.I0, IC55D.I1, IC7A.I, REG-ACU-BUF1A.B7
- new net ACU-DATA7: IC57A.I0, IC58A.I1, IC8A.I, REG-ACU-BUF1A.B8
- new net ALU-EO: ALU-BUFA.G, REG-ACU-BUF1A.G
- new net MBR-DATA0: IC35D.I0, IC37D.I1, REG-MBR-BUF1A.B1
- new net MBR-DATA1: IC38A.I1, IC39A.I0, REG-MBR-BUF1A.B2
- new net MBR-DATA2: IC41D.I1, IC42D.I0, REG-MBR-BUF1A.B3
- new net MBR-DATA3: IC44A.I1, IC45A.I0, REG-MBR-BUF1A.B4
- new net MBR-DATA4: IC48D.I0, IC50D.I1, REG-MBR-BUF1A.B5
- new net MBR-DATA5: IC51A.I1, IC52A.I0, REG-MBR-BUF1A.B6
- new net MBR-DATA6: IC54D.I1, IC55D.I0, REG-MBR-BUF1A.B7
- new net MBR-DATA7: IC57A.I1, IC58A.I0, REG-MBR-BUF1A.B8
- net REG-ACU-DATA0: now also REG-ACU-BUF1A.A1; no longer IC1A.I, IC35D.I1, IC37D.I0
- net REG-ACU-DATA1: now also REG-ACU-BUF1A.A2; no longer IC2A.I, IC38A.I0, IC39A.I1
- net REG-ACU-DATA2: now also REG-ACU-BUF1A.A3; no longer IC3A.I, IC41D.I0, IC42D.I1
- net REG-ACU-DATA3: now also REG-ACU-BUF1A.A4; no longer IC44A.I0, IC45A.I1, IC4A.I
- net REG-ACU-DATA4: now also LED30.A, REG-ACU-BUF0A.A5, REG-ACU-BUF1A.A5; no longer IC48D.I1, IC50D.I0, IC5A.I
- net REG-ACU-DATA5: now also REG-ACU-BUF1A.A6; no longer IC51A.I0, IC52A.I1, IC6A.I
- net REG-ACU-DATA6: now also REG-ACU-BUF1A.A7; no longer IC54D.I0, IC55D.I1, IC7A.I
- net REG-ACU-DATA7: now also LED27.A, REG-ACU-BUF0A.A8, REG-ACU-BUF1A.A8; no longer IC57A.I0, IC58A.I1, IC8A.I
- net REG-MBR-DATA0: now also REG-MBR-BUF1A.A1; no longer IC35D.I0, IC37D.I1
- net REG-MBR-DATA1: now also REG-MBR-BUF1A.A2; no longer IC38A.I1, IC39A.I0
- net REG-MBR-DATA2: now also REG-MBR-BUF1A.A3; no longer IC41D.I1, IC42D.I0
- net REG-MBR-DATA3: now also REG-MBR-BUF1A.A4; no longer IC44A.I1, IC45A.I0
- net REG-MBR-DATA4: now also REG-MBR-BUF1A.A5; no longer IC48D.I0, IC50D.I1
- net REG-MBR-DATA5: now also REG-MBR-BUF1A.A6; no longer IC51A.I1, IC52A.I0
- net REG-MBR-DATA6: now also REG-MBR-BUF1A.A7; no longer IC54D.I1, IC55D.I0
- net REG-MBR-DATA7: now also REG-MBR-BUF1A.A8; no longer IC57A.I1, IC58A.I0
- net VCC: now also REG-ACU-BUF1A.DIR, REG-MBR-BUF1A.DIR
Other:
- moved on the sheet: 4BIT-FULL-ADDER-2, 4BIT-FULL-ADDER-3, ALU-BUF, C1, C2, CLK, DUAL-4X1-MUX-0, DUAL-4X1-MUX-1, DUAL-4X1-MUX-2, DUAL-4X1-MUX-3, Q1, Q2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

Commit message: Added control unit, reset circuit and flag reg to the main schema of the system
Parts:
- added 74LS161N: 74160N, 74xx-eu:74160N
- added AT28C16-0, AT28C16-1, AT28C16-2, AT28C16-3: (no value), memory:2816
- added IC10: 74LS04N, 74xx-eu:74LS04N
- added IC11: 74154N, 74xx-eu:74154N
- added IC9: 74ALS00N, 74xx-eu:74ALS00N
- added LED90, LED91, LED92, LED93, LED94, LED95, LED96, LED97, LED98, LED99: (no value), led:LED5MM
- added R4: (no value), resistor:R-EU_0204/5
- added S3: (no value), switch-omron:10-XX
Connections:
- net PCH-IN renamed PCH-I
- net REG-IO3-LOAD-IN renamed IO3-I
- net REG-IO3-LOAD-OUT renamed IO3-O
- removed net A: DUAL-4X1-MUX-0A.A, DUAL-4X1-MUX-1A.A, DUAL-4X1-MUX-2A.A, DUAL-4X1-MUX-3A.A
- removed net B: DUAL-4X1-MUX-0A.B, DUAL-4X1-MUX-1A.B, DUAL-4X1-MUX-2A.B, DUAL-4X1-MUX-3A.B
- removed net C: 4BIT-FULL-ADDER-2A.C0, IC46A.I0, IC46B.I0, IC46C.I0, IC46D.I0, IC47A.I0, IC47B.I0, IC47C.I0, IC47D.I0
- removed net COUNTER-EN: 74LS161N-0A.ENP, 74LS161N-0A.ENT, 74LS161N-1A.ENP, 74LS161N-2A.ENP, 74LS161N-3A.ENP
- removed net COUNTER-RST: 74LS161N-0A.CLR, 74LS161N-1A.CLR, 74LS161N-2A.CLR, 74LS161N-3A.CLR, RST-INVERTERA.O
- removed net CS-EN: CHIP-SELECT-REG-0A.G1, CHIP-SELECT-REG-0A.G2
- removed net PCH-OUT: PC-BUF-HA.G
- removed net PCL-IN: 74LS161N-0A.LD, 74LS161N-1A.LD
- removed net PCL-OUT: PC-BUF-LA.G
- removed net PR-LOAD: PAGE-ADDR-REG-0A.G1, PAGE-ADDR-REG-0A.G2
- removed net RD: MEMORY-0-8KX8-6264.!OE, MEMORY-1-8KX8-6264.!OE, MEMORY-2-8KX8-6264.!OE, MEMORY-3-8KX8-6264.!OE
- removed net REG-ACU-LOAD-IN: REG-ACU-HA.G1, REG-ACU-HA.G2, REG-ACU-LA.G1, REG-ACU-LA.G2
- removed net REG-IO0-LOAD-IN: REG-IO0-HA.G1, REG-IO0-HA.G2, REG-IO0-LA.G1, REG-IO0-LA.G2
- removed net REG-IO0-LOAD-OUT: REG-IO0-BUFA.G
- removed net REG-IO1-LOAD-IN: REG-IO1-HA.G1, REG-IO1-HA.G2, REG-IO1-LA.G1, REG-IO1-LA.G2
- removed net REG-IO1-LOAD-OUT: REG-IO1-BUFA.G
- removed net REG-IO2-LOAD-IN: REG-IO2-HA.G1, REG-IO2-HA.G2, REG-IO2-LA.G1, REG-IO2-LA.G2
- removed net REG-IO2-LOAD-OUT: REG-IO2-BUFA.G
- removed net REG-IR-LOAD-IN: REG-IR-HA.G1, REG-IR-HA.G2, REG-IR-LA.G1, REG-IR-LA.G2
- removed net REG-IR-LOAD-OUT: REG-IR-BUFA.G
- removed net REG-MAR-LOAD-IN: REG-MAR-HA.G1, REG-MAR-HA.G2, REG-MAR-LA.G1, REG-MAR-LA.G2
- removed net REG-MAR-LOAD-OUT: REG-MAR-BUFA.G
- removed net REG-MBR-LOAD-IN: REG-MBR-HA.G1, REG-MBR-HA.G2, REG-MBR-LA.G1, REG-MBR-LA.G2
- removed net REG-MBR-LOAD-OUT: REG-MBR-BUF0A.G
- removed net REG-SC-LOAD-OUT: REG-ACU-BUF0A.G
- removed net WR: MEM-BUFA.DIR, MEMORY-0-8KX8-6264.!WE, MEMORY-1-8KX8-6264.!WE, MEMORY-2-8KX8-6264.!WE, MEMORY-3-8KX8-6264.!WE
- new net ACU-I: AT28C16-1A.D5, REG-ACU-HA.G1, REG-ACU-HA.G2, REG-ACU-LA.G1, REG-ACU-LA.G2
- new net ACU-O: AT28C16-2A.D4, REG-ACU-BUF0A.G
- new net ALU-A: AT28C16-1A.D1, DUAL-4X1-MUX-0A.A, DUAL-4X1-MUX-1A.A, DUAL-4X1-MUX-2A.A, DUAL-4X1-MUX-3A.A
- new net ALU-B: AT28C16-1A.D2, DUAL-4X1-MUX-0A.B, DUAL-4X1-MUX-1A.B, DUAL-4X1-MUX-2A.B, DUAL-4X1-MUX-3A.B
- new net ALU-C: 4BIT-FULL-ADDER-2A.C0, AT28C16-1A.D3, IC46A.I0, IC46B.I0, IC46C.I0, IC46D.I0, IC47A.I0, IC47B.I0, IC47C.I0, IC47D.I0
- new net ALU-O: ALU-BUFA.G, AT28C16-1A.D0
- new net CF: AT28C16-0A.A4, AT28C16-1A.A4, AT28C16-2A.A4, AT28C16-3A.A4
- new net CMD0: AT28C16-0A.A7, AT28C16-1A.A7, AT28C16-2A.A7, AT28C16-3A.A7
- new net CMD1: AT28C16-0A.A8, AT28C16-1A.A8, AT28C16-2A.A8, AT28C16-3A.A8
- new net CMD2: AT28C16-0A.A9, AT28C16-1A.A9, AT28C16-2A.A9, AT28C16-3A.A9
- new net CMD3: AT28C16-0A.A10, AT28C16-1A.A10, AT28C16-2A.A10, AT28C16-3A.A10
- new net CS-I: AT28C16-3A.D4, CHIP-SELECT-REG-0A.G1, CHIP-SELECT-REG-0A.G2
- new net FLAG-I: AT28C16-3A.D5
- new net IO0-I: AT28C16-2A.D1, REG-IO0-HA.G1, REG-IO0-HA.G2, REG-IO0-LA.G1, REG-IO0-LA.G2
- new net IO0-O: AT28C16-3A.D0, REG-IO0-BUFA.G
- new net IO1-I: AT28C16-2A.D2, REG-IO1-HA.G1, REG-IO1-HA.G2, REG-IO1-LA.G1, REG-IO1-LA.G2
- new net IO1-O: AT28C16-3A.D1, REG-IO1-BUFA.G
- new net IO2-I: AT28C16-2A.D3, REG-IO2-HA.G1, REG-IO2-HA.G2, REG-IO2-LA.G1, REG-IO2-LA.G2
- new net IO2-O: AT28C16-3A.D2, REG-IO2-BUFA.G
- new net IR-I: AT28C16-1A.D7, REG-IR-HA.G1, REG-IR-HA.G2, REG-IR-LA.G1, REG-IR-LA.G2
- new net IR-O: AT28C16-2A.D6, REG-IR-BUFA.G
- new net MAR-I: AT28C16-1A.D6, REG-MAR-HA.G1, REG-MAR-HA.G2, REG-MAR-LA.G1, REG-MAR-LA.G2
- new net MAR-O: AT28C16-2A.D5, REG-MAR-BUFA.G
- new net MBR-I: AT28C16-2A.D0, REG-MBR-HA.G1, REG-MBR-HA.G2, REG-MBR-LA.G1, REG-MBR-LA.G2
- new net MBR-O: AT28C16-2A.D7, REG-MBR-BUF0A.G
- new net MRD: AT28C16-0A.D5, MEMORY-0-8KX8-6264.!OE, MEMORY-1-8KX8-6264.!OE, MEMORY-2-8KX8-6264.!OE, MEMORY-3-8KX8-6264.!OE
- new net MWR: AT28C16-0A.D4, MEM-BUFA.DIR, MEMORY-0-8KX8-6264.!WE, MEMORY-1-8KX8-6264.!WE, MEMORY-2-8KX8-6264.!WE, MEMORY-3-8KX8-6264.!WE
- new net N$10: IC9C.O, IC9D.I0, IC9D.I1
- new net N$11: IC11A.0, LED90.A
- new net N$12: IC11A.1, LED91.A
- new net N$13: IC11A.2, LED92.A
- new net N$14: IC11A.3, LED93.A
- new net N$15: IC11A.4, LED94.A
- new net N$16: IC11A.5, LED95.A
- new net N$17: IC11A.6, LED96.A
- new net N$18: IC11A.7, LED97.A
- new net N$19: IC11A.8, LED98.A
- new net N$20: IC11A.9, LED99.A
- new net N$4: IC9A.I0, IC9A.I1, R4.2, S3.S
- new net PC-EN: 74LS161N-0A.ENP, 74LS161N-0A.ENT, 74LS161N-1A.ENP, 74LS161N-2A.ENP, 74LS161N-3A.ENP, AT28C16-0A.D6
- new net PC-I: AT28C16-0A.D7
- new net PCH-O: AT28C16-0A.D1, PC-BUF-HA.G
- new net PCL-I: 74LS161N-0A.LD, 74LS161N-1A.LD, AT28C16-3A.D3
- new net PCL-O: AT28C16-0A.D0, PC-BUF-LA.G
- new net PR-I: AT28C16-0A.D2, PAGE-ADDR-REG-0A.G1, PAGE-ADDR-REG-0A.G2
- new net RST-H: IC9B.O, REG-ACU-HA.CLR, REG-ACU-LA.CLR, REG-IO0-HA.CLR, REG-IO0-LA.CLR, REG-IO1-HA.CLR, REG-IO1-LA.CLR, REG-IO2-HA.CLR, REG-IO2-LA.CLR, REG-IO3-HA.CLR, REG-IO3-LA.CLR, REG-IR-HA.CLR, REG-IR-LA.CLR, REG-MAR-HA.CLR, REG-MAR-LA.CLR, REG-MBR-HA.CLR, REG-MBR-LA.CLR
- new net RST-L: 74LS161N-0A.CLR, 74LS161N-1A.CLR, 74LS161N-2A.CLR, 74LS161N-3A.CLR, IC9A.O, IC9B.I0, IC9B.I1, IC9C.I0, RST-INVERTERA.O
- new net RST-USTEP: 74LS161NA.CLR, IC11A.10, IC9D.O
- new net SF: AT28C16-0A.A5, AT28C16-1A.A5, AT28C16-2A.A5, AT28C16-3A.A5
- new net USTEP: IC9C.I1
- new net USTEP-A: 74LS161NA.QA, AT28C16-0A.A0, AT28C16-1A.A0, AT28C16-2A.A0, AT28C16-3A.A0, IC11A.A
- new net USTEP-B: 74LS161NA.QB, AT28C16-0A.A1, AT28C16-1A.A1, AT28C16-2A.A1, AT28C16-3A.A1, IC11A.B
- new net USTEP-C: 74LS161NA.QC, AT28C16-0A.A2, AT28C16-1A.A2, AT28C16-2A.A2, AT28C16-3A.A2, IC11A.C
- new net USTEP-D: 74LS161NA.QD, AT28C16-0A.A3, AT28C16-1A.A3, AT28C16-2A.A3, AT28C16-3A.A3, IC11A.D
- new net ZF: AT28C16-0A.A6, AT28C16-1A.A6, AT28C16-2A.A6, AT28C16-3A.A6
- net ALU-EO: no longer ALU-BUFA.G
- net CLK-SIG: now also 74LS161NA.CLK, IC10A.I, IC10A.O
- net GND: now also 74LS161NA.A, 74LS161NA.B, 74LS161NA.C, 74LS161NA.D, 74LS161NA.RCO, AT28C16-0A.!CE, AT28C16-0A.!OE, AT28C16-1A.!CE, AT28C16-1A.!OE, AT28C16-2A.!CE, AT28C16-2A.!OE, AT28C16-3A.!CE, AT28C16-3A.!OE, AT28C16-3A.D6, AT28C16-3A.D7, IC11A.11, IC11A.12, IC11A.13, IC11A.14, IC11A.15, IC11A.G1, IC11A.G2, LED90.C, LED91.C, LED92.C, LED93.C, LED94.C, LED95.C, LED96.C, LED97.C, LED98.C, LED99.C, R4.1, S3.P1, S3.S1; no longer REG-ACU-HA.CLR, REG-ACU-LA.CLR, REG-IO0-HA.CLR, REG-IO0-LA.CLR, REG-IO1-HA.CLR, REG-IO1-LA.CLR, REG-IO2-HA.CLR, REG-IO2-LA.CLR, REG-IO3-HA.CLR, REG-IO3-LA.CLR, REG-IR-HA.CLR, REG-IR-LA.CLR, REG-MAR-HA.CLR, REG-MAR-LA.CLR, REG-MBR-HA.CLR, REG-MBR-LA.CLR
- net HLT: now also AT28C16-1A.D4
- net MRQ: now also AT28C16-0A.D3
- net VCC: now also 74LS161NA.ENP, 74LS161NA.ENT, 74LS161NA.LD, AT28C16-0A.!WE, AT28C16-1A.!WE, AT28C16-2A.!WE, AT28C16-3A.!WE, S3.P
Other:
- note added: "CONTROL UNIT"
- note added: "RESET CIRCUIT"
