File: alu/schema/alu.sch (EAGLE design)
At the start: 40 parts, among them IC1 74LS32N, IC10 74LS32N, IC11 74LS08N, IC12 74LS32N, IC13 74LS06N, IC14 74LS08N, IC15 74LS32N, IC16 74LS08N, IC17 74LS86N, IC18 74LS86N, IC19 74LS32N, IC2 74LS06N, IC20 74LS06N, IC21 74LS08N, IC22 74LS08N, IC23 74LS32N, IC24 74LS06N, IC25 74LS08N, IC26 74LS32N, IC27 74LS08N, IC28 74LS32N, IC29 74LS08N, IC3 74LS08N, IC30 74LS32N, IC31 74LS06N, IC32 74LS08N, IC33 74LS32N, IC34 74LS245N, IC4 74LS08N, IC5 74LS32N, IC6 74LS06N, IC7 74LS08N, IC8 74LS32N, IC9 74LS08N

Commit message: Added fixes for ALU schema
Connections:
- removed net ADD0-B0-IN: IC1D.I0, IC3D.I1
- removed net ADD0-B1-IN: IC4A.I1, IC5A.I0
- removed net ADD0-B2-IN: IC7D.I1, IC8D.I0
- removed net ADD0-B3-IN: IC14A.I1, IC15A.I0
- removed net ADD1-B4-IN: IC19D.I0, IC21D.I1
- removed net ADD1-B5-IN: IC22A.I1, IC23A.I0
- removed net ADD1-B6-IN: IC25D.I1, IC26D.I0
- removed net ADD1-B7-IN: IC32A.I1, IC33A.I0
- net ADD0-A0-IN: no longer IC1D.I1, IC2B.I, IC3D.I0
- net ADD0-A1-IN: no longer IC2C.I, IC4A.I0, IC5A.I1
- net ADD0-A2-IN: no longer IC6B.I, IC7D.I0, IC8D.I1
- net ADD0-A3-IN: no longer IC13B.I, IC14A.I0, IC15A.I1
- net ADD1-A4-IN: no longer IC19D.I1, IC20B.I, IC21D.I0
- net ADD1-A5-IN: no longer IC20C.I, IC22A.I0, IC23A.I1
- net ADD1-A6-IN: no longer IC24B.I, IC25D.I0, IC26D.I1
- net ADD1-A7-IN: no longer IC31B.I, IC32A.I0, IC33A.I1
- net ALU-A0-IN: now also IC1D.I1, IC2B.I, IC3D.I0
- net ALU-A1-IN: now also IC2C.I, IC4A.I0, IC5A.I1
- net ALU-A2-IN: now also IC6B.I, IC7D.I0, IC8D.I1
- net ALU-A3-IN: now also IC13B.I, IC14A.I0, IC15A.I1
- net ALU-A4-IN: now also IC19D.I1, IC20B.I, IC21D.I0
- net ALU-A5-IN: now also IC20C.I, IC22A.I0, IC23A.I1
- net ALU-A6-IN: now also IC24B.I, IC25D.I0, IC26D.I1
- net ALU-A7-IN: now also IC31B.I, IC32A.I0, IC33A.I1
- net ALU-B0-IN: now also IC1D.I0, IC3D.I1
- net ALU-B1-IN: now also IC4A.I1, IC5A.I0
- net ALU-B2-IN: now also IC7D.I1, IC8D.I0
- net ALU-B3-IN: now also IC14A.I1, IC15A.I0
- net ALU-B4-IN: now also IC19D.I0, IC21D.I1
- net ALU-B5-IN: now also IC22A.I1, IC23A.I0
- net ALU-B6-IN: now also IC25D.I1, IC26D.I0
- net ALU-B7-IN: now also IC32A.I1, IC33A.I0
- net GND: now also DUAL-4X1-MUX-0A.1G, DUAL-4X1-MUX-0A.2G, DUAL-4X1-MUX-1A.1G, DUAL-4X1-MUX-1A.2G, DUAL-4X1-MUX-2A.1G, DUAL-4X1-MUX-2A.2G, DUAL-4X1-MUX-3A.1G, DUAL-4X1-MUX-3A.2G
- net VCC: no longer DUAL-4X1-MUX-0A.1G, DUAL-4X1-MUX-0A.2G, DUAL-4X1-MUX-1A.1G, DUAL-4X1-MUX-1A.2G, DUAL-4X1-MUX-2A.1G, DUAL-4X1-MUX-2A.2G, DUAL-4X1-MUX-3A.1G, DUAL-4X1-MUX-3A.2G

Commit message: Changed 74LS06N which is inverter with open collector outputs into 74LS04N with standard outputs
Parts:
- removed 4BIT-FULL-ADDER-0, 4BIT-FULL-ADDER-1: 74LS283N, 74xx-eu:74LS283N
- removed IC10, IC12, IC15, IC19, IC23, IC26, IC28, IC30, IC33: 74LS32N, 74xx-eu:74LS32N
- removed IC11, IC14, IC16, IC21, IC22, IC25, IC27, IC29, IC32, IC9: 74LS08N, 74xx-eu:74LS08N
- removed IC13, IC20, IC24, IC31: 74LS06N, 74xx-eu:74LS06N
- removed IC17, IC18: 74LS86N, 74xx-eu:74LS86N
- removed IC34: 74LS245N, 74xx-eu:74LS245N
- added 4BIT-FULL-ADDER-2, 4BIT-FULL-ADDER-3: 74LS283N, 74xx-eu:74LS283N
- added IC35, IC39, IC42, IC45, IC48, IC52, IC55, IC58: 74LS32N, 74xx-eu:74LS32N
- added IC37, IC38, IC41, IC44, IC50, IC51, IC54, IC57: 74LS08N, 74xx-eu:74LS08N
- added IC46, IC47: 74LS86N, 74xx-eu:74LS86N
- added IC59: 74LS245N, 74xx-eu:74LS245N
- IC1, IC5, IC8: value 74LS32N -> 74LS04N; device 74xx-eu:74LS32N -> 74xx-eu:74LS04N
- IC2, IC6: value 74LS06N -> 74LS04N; device 74xx-eu:74LS06N -> 74xx-eu:74LS04N
- IC3, IC4, IC7: value 74LS08N -> 74LS04N; device 74xx-eu:74LS08N -> 74xx-eu:74LS04N
Connections:
- removed net ADD0-S0-OUT: 4BIT-FULL-ADDER-0A.S1, IC3B.I1
- removed net ADD0-S1-OUT: 4BIT-FULL-ADDER-0A.S2, IC3C.I1
- removed net ADD0-S2-OUT: 4BIT-FULL-ADDER-0A.S3, IC9B.I1
- removed net ADD0-S3-OUT: 4BIT-FULL-ADDER-0A.S4, IC11C.I1
- removed net ADD1-S4-OUT: 4BIT-FULL-ADDER-1A.S1, IC21B.I1
- removed net ADD1-S5-OUT: 4BIT-FULL-ADDER-1A.S2, IC21C.I1
- removed net ADD1-S6-OUT: 4BIT-FULL-ADDER-1A.S3, IC27B.I1
- removed net ADD1-S7-OUT: 4BIT-FULL-ADDER-1A.S4, IC29C.I1
- removed net MUX-C0: IC11C.I0, IC16A.I0, IC21B.I0, IC21C.I0, IC29C.I0, IC2A.O, IC3A.I0, IC3B.I0, IC3C.I0
- removed net MUX0-C0: IC27B.I0, IC9B.I0
- removed net N$10: IC10B.I0, IC9B.O
- removed net N$11: DUAL-4X1-MUX-1A.1Y, IC10B.I1
- removed net N$12: DUAL-4X1-MUX-1A.2Y, IC12B.I0
- removed net N$13: DUAL-4X1-MUX-0A.1Y, IC1B.I1
- removed net N$14: IC1C.I1, IC3C.O
- removed net N$15: IC11C.O, IC12B.I1
- removed net N$16: 4BIT-FULL-ADDER-1A.C0, IC3A.O
- removed net N$18: DUAL-4X1-MUX-2A.1Y, IC19B.I1
- removed net N$19: DUAL-4X1-MUX-2A.2Y, IC19C.I0
- removed net N$20: IC19C.I1, IC21C.O
- removed net N$21: IC27B.O, IC28B.I0
- removed net N$22: DUAL-4X1-MUX-3A.1Y, IC28B.I1
- removed net N$23: DUAL-4X1-MUX-3A.2Y, IC30B.I0
- removed net N$24: IC29C.O, IC30B.I1
- removed net N$5: IC1A.O, IC2A.I
- removed net N$7: 4BIT-FULL-ADDER-0A.C4, IC3A.I1
- removed net N$8: DUAL-4X1-MUX-0A.2Y, IC1C.I0
- removed net N$9: 4BIT-FULL-ADDER-1A.C4, IC16A.I1
- removed net S0_1_OUT: IC1B.I0, IC3B.O
- removed net S0_1_OUT1: IC19B.I0, IC21B.O
- new net MUX0-1C0-IN: 4BIT-FULL-ADDER-2A.S1, DUAL-4X1-MUX-0A.1C0
- new net MUX0-2C0-IN: 4BIT-FULL-ADDER-2A.S2, DUAL-4X1-MUX-0A.2C0
- new net MUX1-1C0-IN: 4BIT-FULL-ADDER-2A.S3, DUAL-4X1-MUX-1A.1C0
- new net MUX1-2C0-IN: 4BIT-FULL-ADDER-2A.S4, DUAL-4X1-MUX-1A.2C0
- new net MUX2-1C0-IN: 4BIT-FULL-ADDER-3A.S1, DUAL-4X1-MUX-2A.1C0
- new net MUX2-2C0-IN: 4BIT-FULL-ADDER-3A.S2, DUAL-4X1-MUX-2A.2C0
- new net MUX3-1C0-IN: 4BIT-FULL-ADDER-3A.S3, DUAL-4X1-MUX-3A.1C0
- new net MUX3-2C0-IN: 4BIT-FULL-ADDER-3A.S4, DUAL-4X1-MUX-3A.2C0
- new net N$1: 4BIT-FULL-ADDER-2A.C4, 4BIT-FULL-ADDER-3A.C0
- net A: no longer IC1A.I0
- net ADD0-A0-IN: now also 4BIT-FULL-ADDER-2A.A1, IC46A.O; no longer 4BIT-FULL-ADDER-0A.A1, IC17A.O
- net ADD0-A1-IN: now also 4BIT-FULL-ADDER-2A.A2, IC46B.O; no longer 4BIT-FULL-ADDER-0A.A2, IC17B.O
- net ADD0-A2-IN: now also 4BIT-FULL-ADDER-2A.A3, IC46C.O; no longer 4BIT-FULL-ADDER-0A.A3, IC17C.O
- net ADD0-A3-IN: now also 4BIT-FULL-ADDER-2A.A4, IC46D.O; no longer 4BIT-FULL-ADDER-0A.A4, IC17D.O
- net ADD1-A4-IN: now also 4BIT-FULL-ADDER-3A.A1, IC47A.O; no longer 4BIT-FULL-ADDER-1A.A1, IC18A.O
- net ADD1-A5-IN: now also 4BIT-FULL-ADDER-3A.A2, IC47B.O; no longer 4BIT-FULL-ADDER-1A.A2, IC18B.O
- net ADD1-A6-IN: now also 4BIT-FULL-ADDER-3A.A3, IC47C.O; no longer 4BIT-FULL-ADDER-1A.A3, IC18C.O
- net ADD1-A7-IN: now also 4BIT-FULL-ADDER-3A.A4, IC47D.O; no longer 4BIT-FULL-ADDER-1A.A4, IC18D.O
- net ALU-A0-IN: now also IC1A.I, IC35D.I1, IC37D.I0, IC46A.I1; no longer IC17A.I1, IC1D.I1, IC2B.I, IC3D.I0
- net ALU-A1-IN: now also IC2A.I, IC38A.I0, IC39A.I1, IC46B.I1; no longer IC17B.I1, IC2C.I, IC4A.I0, IC5A.I1
- net ALU-A2-IN: now also IC3A.I, IC41D.I0, IC42D.I1, IC46C.I1; no longer IC17C.I1, IC6B.I, IC7D.I0, IC8D.I1
- net ALU-A3-IN: now also IC44A.I0, IC45A.I1, IC46D.I1, IC4A.I; no longer IC13B.I, IC14A.I0, IC15A.I1, IC17D.I1
- net ALU-A4-IN: now also IC47A.I1, IC48D.I1, IC50D.I0, IC5A.I; no longer IC18A.I1, IC19D.I1, IC20B.I, IC21D.I0
- net ALU-A5-IN: now also IC47B.I1, IC51A.I0, IC52A.I1, IC6A.I; no longer IC18B.I1, IC20C.I, IC22A.I0, IC23A.I1
- net ALU-A6-IN: now also IC47C.I1, IC54D.I0, IC55D.I1, IC7A.I; no longer IC18C.I1, IC24B.I, IC25D.I0, IC26D.I1
- net ALU-A7-IN: now also IC47D.I1, IC57A.I0, IC58A.I1, IC8A.I; no longer IC18D.I1, IC31B.I, IC32A.I0, IC33A.I1
- net ALU-B0-IN: now also 4BIT-FULL-ADDER-2A.B1, IC35D.I0, IC37D.I1; no longer 4BIT-FULL-ADDER-0A.B1, IC1D.I0, IC3D.I1
- net ALU-B1-IN: now also 4BIT-FULL-ADDER-2A.B2, IC38A.I1, IC39A.I0; no longer 4BIT-FULL-ADDER-0A.B2, IC4A.I1, IC5A.I0
- net ALU-B2-IN: now also 4BIT-FULL-ADDER-2A.B3, IC41D.I1, IC42D.I0; no longer 4BIT-FULL-ADDER-0A.B3, IC7D.I1, IC8D.I0
- net ALU-B3-IN: now also 4BIT-FULL-ADDER-2A.B4, IC44A.I1, IC45A.I0; no longer 4BIT-FULL-ADDER-0A.B4, IC14A.I1, IC15A.I0
- net ALU-B4-IN: now also 4BIT-FULL-ADDER-3A.B1, IC48D.I0, IC50D.I1; no longer 4BIT-FULL-ADDER-1A.B1, IC19D.I0, IC21D.I1
- net ALU-B5-IN: now also 4BIT-FULL-ADDER-3A.B2, IC51A.I1, IC52A.I0; no longer 4BIT-FULL-ADDER-1A.B2, IC22A.I1, IC23A.I0
- net ALU-B6-IN: now also 4BIT-FULL-ADDER-3A.B3, IC54D.I1, IC55D.I0; no longer 4BIT-FULL-ADDER-1A.B3, IC25D.I1, IC26D.I0
- net ALU-B7-IN: now also 4BIT-FULL-ADDER-3A.B4, IC57A.I1, IC58A.I0; no longer 4BIT-FULL-ADDER-1A.B4, IC32A.I1, IC33A.I0
- net ALU-C0-BUS-IN: now also IC59A.B1; no longer IC34A.B1
- net ALU-C0-OUT: now also DUAL-4X1-MUX-0A.1Y, IC59A.A1; no longer IC1B.O, IC34A.A1
- net ALU-C1-BUS-IN: now also IC59A.B2; no longer IC34A.B2
- net ALU-C1-OUT: now also DUAL-4X1-MUX-0A.2Y, IC59A.A2; no longer IC1C.O, IC34A.A2
- net ALU-C2-BUS-IN: now also IC59A.B3; no longer IC34A.B3
- net ALU-C2-OUT: now also DUAL-4X1-MUX-1A.1Y, IC59A.A3; no longer IC10B.O, IC34A.A3
- net ALU-C3-BUS-IN: now also IC59A.B4; no longer IC34A.B4
- net ALU-C3-OUT: now also DUAL-4X1-MUX-1A.2Y, IC59A.A4; no longer IC12B.O, IC34A.A4
- net ALU-C4-BUS-IN: now also IC59A.B5; no longer IC34A.B5
- net ALU-C4-OUT: now also DUAL-4X1-MUX-2A.1Y, IC59A.A5; no longer IC19B.O, IC34A.A5
- net ALU-C5-BUS-IN: now also IC59A.B6; no longer IC34A.B6
- net ALU-C5-OUT: now also DUAL-4X1-MUX-2A.2Y, IC59A.A6; no longer IC19C.O, IC34A.A6
- net ALU-C6-BUS-IN: now also IC59A.B7; no longer IC34A.B7
- net ALU-C6-OUT: now also DUAL-4X1-MUX-3A.1Y, IC59A.A7; no longer IC28B.O, IC34A.A7
- net ALU-C7-BUS-IN: now also IC59A.B8; no longer IC34A.B8
- net ALU-C7-OUT: now also DUAL-4X1-MUX-3A.2Y, IC59A.A8; no longer IC30B.O, IC34A.A8
- net ALU_EO: now also IC59A.G; no longer IC34A.G
- net B: no longer IC1A.I1
- net C: now also 4BIT-FULL-ADDER-2A.C0, IC46A.I0, IC46B.I0, IC46C.I0, IC46D.I0, IC47A.I0, IC47B.I0, IC47C.I0, IC47D.I0; no longer 4BIT-FULL-ADDER-0A.C0, IC17A.I0, IC17B.I0, IC17C.I0, IC17D.I0, IC18A.I0, IC18B.I0, IC18C.I0, IC18D.I0
- net CARRY-1: now also 4BIT-FULL-ADDER-3A.C4; no longer IC16A.O
- net GND: no longer DUAL-4X1-MUX-0A.1C0, DUAL-4X1-MUX-0A.2C0, DUAL-4X1-MUX-1A.1C0, DUAL-4X1-MUX-1A.2C0, DUAL-4X1-MUX-2A.1C0, DUAL-4X1-MUX-2A.2C0, DUAL-4X1-MUX-3A.1C0, DUAL-4X1-MUX-3A.2C0
- net MUX0-1C1-IN: now also IC35D.O; no longer IC1D.O
- net MUX0-1C2-IN: now also IC1A.O; no longer IC2B.O
- net MUX0-1C3-IN: now also IC37D.O; no longer IC3D.O
- net MUX0-2C1-IN: now also IC39A.O; no longer IC5A.O
- net MUX0-2C2-IN: now also IC2A.O; no longer IC2C.O
- net MUX0-2C3-IN: now also IC38A.O; no longer IC4A.O
- net MUX1-1C1-IN: now also IC42D.O; no longer IC8D.O
- net MUX1-1C2-IN: now also IC3A.O; no longer IC6B.O
- net MUX1-1C3-IN: now also IC41D.O; no longer IC7D.O
- net MUX1-2C1-IN: now also IC45A.O; no longer IC15A.O
- net MUX1-2C2-IN: now also IC4A.O; no longer IC13B.O
- net MUX1-2C3-IN: now also IC44A.O; no longer IC14A.O
- net MUX2-1C1-IN: now also IC48D.O; no longer IC19D.O
- net MUX2-1C2-IN: now also IC5A.O; no longer IC20B.O
- net MUX2-1C3-IN: now also IC50D.O; no longer IC21D.O
- net MUX2-2C1-IN: now also IC52A.O; no longer IC23A.O
- net MUX2-2C2-IN: now also IC6A.O; no longer IC20C.O
- net MUX2-2C3-IN: now also IC51A.O; no longer IC22A.O
- net MUX3-1C1-IN: now also IC55D.O; no longer IC26D.O
- net MUX3-1C2-IN: now also IC7A.O; no longer IC24B.O
- net MUX3-1C3-IN: now also IC54D.O; no longer IC25D.O
- net MUX4-2C1-IN: now also IC58A.O; no longer IC33A.O
- net MUX4-2C2-IN: now also IC8A.O; no longer IC31B.O
- net MUX4-2C3-IN: now also IC57A.O; no longer IC32A.O
- net VCC: now also IC59A.DIR; no longer IC34A.DIR
Other:
- moved on the sheet: DUAL-4X1-MUX-0, DUAL-4X1-MUX-1, DUAL-4X1-MUX-2, DUAL-4X1-MUX-3, IC2A, IC3A, IC4A

Commit message: Group ALU mux ifaces into the bus
Connections:
- net MUX0-1C0-IN renamed MUX0-1C0
- net MUX0-1C1-IN renamed MUX0-1C1
- net MUX0-1C2-IN renamed MUX0-1C2
- net MUX0-1C3-IN renamed MUX0-1C3
- net MUX0-2C0-IN renamed MUX0-2C0
- net MUX0-2C1-IN renamed MUX0-2C1
- net MUX0-2C2-IN renamed MUX0-2C2
- net MUX0-2C3-IN renamed MUX0-2C3
- net MUX1-1C0-IN renamed MUX1-1C0
- net MUX1-1C1-IN renamed MUX1-1C1
- net MUX1-1C2-IN renamed MUX1-1C2
- net MUX1-1C3-IN renamed MUX1-1C3
- net MUX1-2C0-IN renamed MUX1-2C0
- net MUX2-1C0-IN renamed MUX2-1C0
- net MUX2-1C1-IN renamed MUX2-1C1
- net MUX2-1C2-IN renamed MUX2-1C2
- net MUX2-1C3-IN renamed MUX2-1C3
- net MUX2-2C0-IN renamed MUX2-2C0
- net MUX2-2C1-IN renamed MUX2-2C1
- net MUX2-2C2-IN renamed MUX2-2C2
- net MUX2-2C3-IN renamed MUX2-2C3
- net MUX3-1C0-IN renamed MUX3-1C0
- net MUX3-1C1-IN renamed MUX3-1C1
- net MUX3-1C2-IN renamed MUX3-1C2
- net MUX3-1C3-IN renamed MUX3-1C3
- net MUX3-2C0-IN renamed MUX3-2C0
- net MUX4-2C1-IN renamed MUX3-2C1
- net MUX4-2C2-IN renamed MUX3-2C2
- net MUX4-2C3-IN renamed MUX3-2C3
- new net MUX1-2C1: DUAL-4X1-MUX-1A.2C1
- new net MUX1-2C2: DUAL-4X1-MUX-1A.2C2
- new net MUX1-2C3: DUAL-4X1-MUX-1A.2C3
- net MUX1-2C1-IN: no longer DUAL-4X1-MUX-1A.2C1
- net MUX1-2C2-IN: no longer DUAL-4X1-MUX-1A.2C2
- net MUX1-2C3-IN: no longer DUAL-4X1-MUX-1A.2C3
Other:
- moved on the sheet: IC46A, IC46B, IC46C, IC46D, IC47A, IC47B, IC47C, IC47D
