File: ram/schema/dbg-ram-4x8K.sch (EAGLE design)
At the start: 0 parts

Commit message: Added debug schema for SRAM circuit
Parts:
- added DEMUX-2X4-0: 74LS139N, 74xx-eu:74LS139N
- added IC1, IC2, IC3: 74LS245N, 74xx-eu:74LS245N
- added LED1, LED10, LED11, LED12, LED13, LED14, LED15, LED17, LED18, LED19, LED2, LED20, LED21, LED22, LED23, LED24, LED25, LED3, LED4, LED5, LED6, LED7, LED8, LED9: (no value), led:LED5MM
- added MEMORY-0-8KX8-6264, MEMORY-1-8KX8-6264, MEMORY-2-8KX8-6264, MEMORY-3-8KX8-6264: (no value), memory-hitachi:6264A
- added PAGE-ADDR-REG-0: 74LS173N, 74xx-eu:74LS173N
Connections:
- new net ADDR-A0: IC1A.A5, LED1.A
- new net ADDR-A1: IC1A.A6, LED2.A
- new net ADDR-A2: IC1A.A7, LED3.A
- new net ADDR-A3: IC1A.A8, LED4.A
- new net ADDR-A4: IC2A.A1, LED5.A
- new net ADDR-A5: IC2A.A2, LED6.A
- new net ADDR-A6: IC2A.A3, LED10.A
- new net ADDR-A7: IC2A.A4, LED7.A
- new net ADDR-A8: IC2A.A5, LED8.A
- new net ADDR-A9: IC2A.A6, LED9.A
- new net ADDR-B10: DEMUX-2X4-0A.A, IC2A.A7, LED15.A, PAGE-ADDR-REG-0A.Q1
- new net ADDR-B11: DEMUX-2X4-0A.B, IC2A.A8, LED17.A, PAGE-ADDR-REG-0A.Q2
- new net ADDR-B12: PAGE-ADDR-REG-0A.Q3
- new net ADDR-C0: IC1A.B5, MEMORY-0-8KX8-6264.A0, MEMORY-1-8KX8-6264.A0, MEMORY-2-8KX8-6264.A0, MEMORY-3-8KX8-6264.A0
- new net ADDR-C1: IC1A.B6, MEMORY-0-8KX8-6264.A1, MEMORY-1-8KX8-6264.A1, MEMORY-2-8KX8-6264.A1, MEMORY-3-8KX8-6264.A1
- new net ADDR-C2: IC1A.B7, MEMORY-0-8KX8-6264.A2, MEMORY-1-8KX8-6264.A2, MEMORY-2-8KX8-6264.A2, MEMORY-3-8KX8-6264.A2
- new net ADDR-C3: IC1A.B8, MEMORY-0-8KX8-6264.A3, MEMORY-1-8KX8-6264.A3, MEMORY-2-8KX8-6264.A3, MEMORY-3-8KX8-6264.A3
- new net ADDR-C4: IC2A.B1, MEMORY-0-8KX8-6264.A4, MEMORY-1-8KX8-6264.A4, MEMORY-2-8KX8-6264.A4, MEMORY-3-8KX8-6264.A4
- new net ADDR-C5: IC2A.B2, MEMORY-0-8KX8-6264.A5, MEMORY-1-8KX8-6264.A5, MEMORY-2-8KX8-6264.A5, MEMORY-3-8KX8-6264.A5
- new net ADDR-C6: IC2A.B3, MEMORY-0-8KX8-6264.A6, MEMORY-1-8KX8-6264.A6, MEMORY-2-8KX8-6264.A6, MEMORY-3-8KX8-6264.A6
- new net ADDR-C7: IC2A.B4, MEMORY-0-8KX8-6264.A7, MEMORY-1-8KX8-6264.A7, MEMORY-2-8KX8-6264.A7, MEMORY-2-8KX8-6264.A8, MEMORY-3-8KX8-6264.A7
- new net ADDR-C8: IC2A.B5, MEMORY-0-8KX8-6264.A8, MEMORY-1-8KX8-6264.A8, MEMORY-3-8KX8-6264.A8
- new net ADDR-C9: IC2A.B6, MEMORY-0-8KX8-6264.A9, MEMORY-1-8KX8-6264.A9, MEMORY-2-8KX8-6264.A9, MEMORY-3-8KX8-6264.A9
- new net ADDR-D10: IC2A.B7, MEMORY-0-8KX8-6264.A10, MEMORY-1-8KX8-6264.A10, MEMORY-2-8KX8-6264.A10, MEMORY-3-8KX8-6264.A10
- new net ADDR-D11: IC2A.B8, MEMORY-0-8KX8-6264.A11, MEMORY-1-8KX8-6264.A11, MEMORY-2-8KX8-6264.A11, MEMORY-3-8KX8-6264.A11
- new net ADDR-D12: MEMORY-0-8KX8-6264.A12, MEMORY-1-8KX8-6264.A12, MEMORY-2-8KX8-6264.A12, MEMORY-3-8KX8-6264.A12
- new net CLK-SIG: PAGE-ADDR-REG-0A.CLK
- new net DATA-A0: IC3A.B1
- new net DATA-A1: IC3A.B2
- new net DATA-A2: IC3A.B3
- new net DATA-A3: IC3A.B4
- new net DATA-A4: IC3A.B5
- new net DATA-A5: IC3A.B6
- new net DATA-A6: IC3A.B7
- new net DATA-A7: IC3A.B8
- new net DATA-B0: IC3A.A1, LED25.A, MEMORY-0-8KX8-6264.I/O1, MEMORY-1-8KX8-6264.I/O1, MEMORY-2-8KX8-6264.I/O1, MEMORY-3-8KX8-6264.I/O1, PAGE-ADDR-REG-0A.D1
- new net DATA-B1: IC3A.A2, LED24.A, MEMORY-0-8KX8-6264.I/O2, MEMORY-1-8KX8-6264.I/O2, MEMORY-2-8KX8-6264.I/O2, MEMORY-3-8KX8-6264.I/O2, PAGE-ADDR-REG-0A.D2
- new net DATA-B2: IC3A.A3, LED23.A, MEMORY-0-8KX8-6264.I/O3, MEMORY-1-8KX8-6264.I/O3, MEMORY-2-8KX8-6264.I/O3, MEMORY-3-8KX8-6264.I/O3, PAGE-ADDR-REG-0A.D3
- new net DATA-B3: IC3A.A4, LED22.A, MEMORY-0-8KX8-6264.I/O4, MEMORY-1-8KX8-6264.I/O4, MEMORY-2-8KX8-6264.I/O4, MEMORY-3-8KX8-6264.I/O4, PAGE-ADDR-REG-0A.D4
- new net DATA-B4: IC3A.A5, LED21.A, MEMORY-0-8KX8-6264.I/O5, MEMORY-1-8KX8-6264.I/O5, MEMORY-2-8KX8-6264.I/O5, MEMORY-3-8KX8-6264.I/O5
- new net DATA-B5: IC3A.A6, LED20.A, MEMORY-0-8KX8-6264.I/O6, MEMORY-1-8KX8-6264.I/O6, MEMORY-2-8KX8-6264.I/O6, MEMORY-3-8KX8-6264.I/O6
- new net DATA-B6: IC3A.A7, LED19.A, MEMORY-0-8KX8-6264.I/O7, MEMORY-1-8KX8-6264.I/O7, MEMORY-2-8KX8-6264.I/O7, MEMORY-3-8KX8-6264.I/O7
- new net DATA-B7: IC3A.A8, LED18.A, MEMORY-0-8KX8-6264.I/O8, MEMORY-1-8KX8-6264.I/O8, MEMORY-2-8KX8-6264.I/O8, MEMORY-3-8KX8-6264.I/O8
- new net GND: IC1A.G, IC2A.G, LED1.C, LED10.C, LED11.C, LED12.C, LED13.C, LED14.C, LED15.C, LED17.C, LED18.C, LED19.C, LED2.C, LED20.C, LED21.C, LED22.C, LED23.C, LED24.C, LED25.C, LED3.C, LED4.C, LED5.C, LED6.C, LED7.C, LED8.C, LED9.C, MEMORY-0-8KX8-6264.VSS, MEMORY-1-8KX8-6264.VSS, MEMORY-2-8KX8-6264.VSS, MEMORY-3-8KX8-6264.VSS, PAGE-ADDR-REG-0A.CLR, PAGE-ADDR-REG-0A.M, PAGE-ADDR-REG-0A.N, PAGE-ADDR-REG-0A.Q4
- new net MRQ: DEMUX-2X4-0A.G, IC3A.G
- new net PAGE-EN-A0: DEMUX-2X4-0A.Y0, IC1A.A1, LED11.A
- new net PAGE-EN-A1: DEMUX-2X4-0A.Y1, IC1A.A2, LED12.A
- new net PAGE-EN-A2: DEMUX-2X4-0A.Y2, IC1A.A3, LED13.A
- new net PAGE-EN-A3: DEMUX-2X4-0A.Y3, IC1A.A4, LED14.A
- new net PAGE-EN-B0: IC1A.B1, MEMORY-0-8KX8-6264.!CS1
- new net PAGE-EN-B1: IC1A.B2, MEMORY-1-8KX8-6264.!CS1
- new net PAGE-EN-B2: IC1A.B3, MEMORY-2-8KX8-6264.!CS1
- new net PAGE-EN-B3: IC1A.B4, MEMORY-3-8KX8-6264.!CS1
- new net PR-LOAD: PAGE-ADDR-REG-0A.G1, PAGE-ADDR-REG-0A.G2
- new net RD: MEMORY-0-8KX8-6264.!OE, MEMORY-1-8KX8-6264.!OE, MEMORY-2-8KX8-6264.!OE, MEMORY-3-8KX8-6264.!OE
- new net VCC: IC1A.DIR, IC2A.DIR, MEMORY-0-8KX8-6264.CS2, MEMORY-0-8KX8-6264.VCC, MEMORY-1-8KX8-6264.CS2, MEMORY-1-8KX8-6264.VCC, MEMORY-2-8KX8-6264.CS2, MEMORY-2-8KX8-6264.VCC, MEMORY-3-8KX8-6264.CS2, MEMORY-3-8KX8-6264.VCC
- new net WR: IC3A.DIR, MEMORY-0-8KX8-6264.!WE, MEMORY-1-8KX8-6264.!WE, MEMORY-2-8KX8-6264.!WE, MEMORY-3-8KX8-6264.!WE
Other:
- note added: "SRAM (STATIC RANDOM ACCESS MEMORY) 4x8K"
