File: ram/schema/dbg-ram-4x8K.sch (EAGLE design)
At the start: 33 parts, among them IC1 74LS245N, IC2 74LS245N, IC3 74LS245N

Commit message: Added switch between programing and run modes for SRAM
Parts:
- removed IC1, IC2, IC3: 74LS245N, 74xx-eu:74LS245N
- added ADDR-R/P-SW-0, ADDR-R/P-SW-1, ADDR-R/P-SW-2, ADDR-R/P-SW-3, DATA-R/P-SW-0, DATA-R/P-SW-1: 74LS157N, 74xx-eu:74LS157N
- added BUFFER-0, BUFFER-1, BUFFER-2, BUFFER-3: 74LS245N, 74xx-eu:74LS245N
- added LED16: (no value), led:LED5MM
- added PROG/RUN-ADDR-SW: (no value), special:SW_DIP-12
- added PROG/RUN-DATA-SW: (no value), special:SW_DIP-8
- added SW2, SW3: (no value), special:SW_DIP-1
Connections:
- new net ADDR-P0: ADDR-R/P-SW-0A.1B, PROG/RUN-ADDR-SW.1
- new net ADDR-P1: ADDR-R/P-SW-0A.2B, PROG/RUN-ADDR-SW.2
- new net ADDR-P10: ADDR-R/P-SW-2A.3B, PROG/RUN-ADDR-SW.11
- new net ADDR-P11: ADDR-R/P-SW-2A.4B, PROG/RUN-ADDR-SW.12
- new net ADDR-P12: ADDR-R/P-SW-3A.1B, SW3.1
- new net ADDR-P2: ADDR-R/P-SW-0A.3B, PROG/RUN-ADDR-SW.3
- new net ADDR-P3: ADDR-R/P-SW-0A.4B, PROG/RUN-ADDR-SW.4
- new net ADDR-P4: ADDR-R/P-SW-1A.1B, PROG/RUN-ADDR-SW.5
- new net ADDR-P5: ADDR-R/P-SW-1A.2B, PROG/RUN-ADDR-SW.6
- new net ADDR-P6: ADDR-R/P-SW-1A.3B, PROG/RUN-ADDR-SW.7
- new net ADDR-P7: ADDR-R/P-SW-1A.4B, PROG/RUN-ADDR-SW.8
- new net ADDR-P8: ADDR-R/P-SW-2A.1B, PROG/RUN-ADDR-SW.9
- new net ADDR-P9: ADDR-R/P-SW-2A.2B, PROG/RUN-ADDR-SW.10
- new net ADDR-R0: ADDR-R/P-SW-0A.1A
- new net ADDR-R1: ADDR-R/P-SW-0A.2A
- new net ADDR-R10: ADDR-R/P-SW-2A.3A
- new net ADDR-R11: ADDR-R/P-SW-2A.4A
- new net ADDR-R12: ADDR-R/P-SW-3A.1A
- new net ADDR-R2: ADDR-R/P-SW-0A.3A
- new net ADDR-R3: ADDR-R/P-SW-0A.4A
- new net ADDR-R4: ADDR-R/P-SW-1A.1A
- new net ADDR-R5: ADDR-R/P-SW-1A.2A
- new net ADDR-R6: ADDR-R/P-SW-1A.3A
- new net ADDR-R7: ADDR-R/P-SW-1A.4A
- new net ADDR-R8: ADDR-R/P-SW-2A.1A
- new net ADDR-R9: ADDR-R/P-SW-2A.2A
- new net DATA-P0: DATA-R/P-SW-0A.1B, PROG/RUN-DATA-SW.1
- new net DATA-P1: DATA-R/P-SW-0A.2B, PROG/RUN-DATA-SW.2
- new net DATA-P2: DATA-R/P-SW-0A.3B, PROG/RUN-DATA-SW.3
- new net DATA-P3: DATA-R/P-SW-0A.4B, PROG/RUN-DATA-SW.4
- new net DATA-P4: DATA-R/P-SW-1A.1B, PROG/RUN-DATA-SW.5
- new net DATA-P5: DATA-R/P-SW-1A.2B, PROG/RUN-DATA-SW.6
- new net DATA-P6: DATA-R/P-SW-1A.3B, PROG/RUN-DATA-SW.7
- new net DATA-P7: DATA-R/P-SW-1A.4B, PROG/RUN-DATA-SW.8
- new net DATA-R0: DATA-R/P-SW-0A.1A
- new net DATA-R1: DATA-R/P-SW-0A.2A
- new net DATA-R2: DATA-R/P-SW-0A.3A
- new net DATA-R3: DATA-R/P-SW-0A.4A
- new net DATA-R4: DATA-R/P-SW-1A.1A
- new net DATA-R5: DATA-R/P-SW-1A.2A
- new net DATA-R6: DATA-R/P-SW-1A.3A
- new net DATA-R7: DATA-R/P-SW-1A.4A
- new net PROG/RUN-SW: ADDR-R/P-SW-0A.!A!/B, ADDR-R/P-SW-1A.!A!/B, ADDR-R/P-SW-2A.!A!/B, ADDR-R/P-SW-3A.!A!/B, DATA-R/P-SW-0A.!A!/B, DATA-R/P-SW-1A.!A!/B, SW2.1
- net ADDR-A0: now also ADDR-R/P-SW-0A.1Y, BUFFER-0A.A5; no longer IC1A.A5
- net ADDR-A1: now also ADDR-R/P-SW-0A.2Y, BUFFER-0A.A6; no longer IC1A.A6
- net ADDR-A2: now also ADDR-R/P-SW-0A.3Y, BUFFER-0A.A7; no longer IC1A.A7
- net ADDR-A3: now also ADDR-R/P-SW-0A.4Y, BUFFER-0A.A8; no longer IC1A.A8
- net ADDR-A4: now also ADDR-R/P-SW-1A.1Y, BUFFER-1A.A1; no longer IC2A.A1
- net ADDR-A5: now also ADDR-R/P-SW-1A.2Y, BUFFER-1A.A2; no longer IC2A.A2
- net ADDR-A6: now also ADDR-R/P-SW-1A.3Y, BUFFER-1A.A3; no longer IC2A.A3
- net ADDR-A7: now also ADDR-R/P-SW-1A.4Y, BUFFER-1A.A4; no longer IC2A.A4
- net ADDR-A8: now also ADDR-R/P-SW-2A.1Y, BUFFER-1A.A5; no longer IC2A.A5
- net ADDR-A9: now also ADDR-R/P-SW-2A.2Y, BUFFER-1A.A6; no longer IC2A.A6
- net ADDR-B10: now also ADDR-R/P-SW-2A.3Y, BUFFER-1A.A7; no longer IC2A.A7
- net ADDR-B11: now also ADDR-R/P-SW-2A.4Y, BUFFER-1A.A8; no longer IC2A.A8
- net ADDR-B12: now also ADDR-R/P-SW-3A.1Y, BUFFER-3A.A1, LED16.A
- net ADDR-C0: now also BUFFER-0A.B5; no longer IC1A.B5
- net ADDR-C1: now also BUFFER-0A.B6; no longer IC1A.B6
- net ADDR-C2: now also BUFFER-0A.B7; no longer IC1A.B7
- net ADDR-C3: now also BUFFER-0A.B8; no longer IC1A.B8
- net ADDR-C4: now also BUFFER-1A.B1; no longer IC2A.B1
- net ADDR-C5: now also BUFFER-1A.B2; no longer IC2A.B2
- net ADDR-C6: now also BUFFER-1A.B3; no longer IC2A.B3
- net ADDR-C7: now also BUFFER-1A.B4; no longer IC2A.B4
- net ADDR-C8: now also BUFFER-1A.B5; no longer IC2A.B5
- net ADDR-C9: now also BUFFER-1A.B6; no longer IC2A.B6
- net ADDR-D10: now also BUFFER-1A.B7; no longer IC2A.B7
- net ADDR-D11: now also BUFFER-1A.B8; no longer IC2A.B8
- net ADDR-D12: now also BUFFER-3A.B1
- net DATA-A0: now also BUFFER-2A.B1, DATA-R/P-SW-0A.1Y; no longer IC3A.B1
- net DATA-A1: now also BUFFER-2A.B2, DATA-R/P-SW-0A.2Y; no longer IC3A.B2
- net DATA-A2: now also BUFFER-2A.B3, DATA-R/P-SW-0A.3Y; no longer IC3A.B3
- net DATA-A3: now also BUFFER-2A.B4, DATA-R/P-SW-0A.4Y; no longer IC3A.B4
- net DATA-A4: now also BUFFER-2A.B5, DATA-R/P-SW-1A.1Y; no longer IC3A.B5
- net DATA-A5: now also BUFFER-2A.B6, DATA-R/P-SW-1A.2Y; no longer IC3A.B6
- net DATA-A6: now also BUFFER-2A.B7, DATA-R/P-SW-1A.3Y; no longer IC3A.B7
- net DATA-A7: now also BUFFER-2A.B8, DATA-R/P-SW-1A.4Y; no longer IC3A.B8
- net DATA-B0: now also BUFFER-2A.A1; no longer IC3A.A1
- net DATA-B1: now also BUFFER-2A.A2; no longer IC3A.A2
- net DATA-B2: now also BUFFER-2A.A3; no longer IC3A.A3
- net DATA-B3: now also BUFFER-2A.A4; no longer IC3A.A4
- net DATA-B4: now also BUFFER-2A.A5; no longer IC3A.A5
- net DATA-B5: now also BUFFER-2A.A6; no longer IC3A.A6
- net DATA-B6: now also BUFFER-2A.A7; no longer IC3A.A7
- net DATA-B7: now also BUFFER-2A.A8; no longer IC3A.A8
- net GND: now also ADDR-R/P-SW-0A.G, ADDR-R/P-SW-1A.G, ADDR-R/P-SW-2A.G, ADDR-R/P-SW-3A.G, BUFFER-0A.G, BUFFER-1A.G, BUFFER-3A.G, DATA-R/P-SW-0A.G, DATA-R/P-SW-1A.G, LED16.C, PROG/RUN-ADDR-SW.13, PROG/RUN-ADDR-SW.14, PROG/RUN-ADDR-SW.15, PROG/RUN-ADDR-SW.16, PROG/RUN-ADDR-SW.17, PROG/RUN-ADDR-SW.18, PROG/RUN-ADDR-SW.19, PROG/RUN-ADDR-SW.20, PROG/RUN-ADDR-SW.21, PROG/RUN-ADDR-SW.22, PROG/RUN-ADDR-SW.23, PROG/RUN-ADDR-SW.24, PROG/RUN-DATA-SW.10, PROG/RUN-DATA-SW.11, PROG/RUN-DATA-SW.12, PROG/RUN-DATA-SW.13, PROG/RUN-DATA-SW.14, PROG/RUN-DATA-SW.15, PROG/RUN-DATA-SW.16, PROG/RUN-DATA-SW.9, SW2.2, SW3.2; no longer IC1A.G, IC2A.G
- net MRQ: now also BUFFER-2A.G; no longer IC3A.G
- net PAGE-EN-A0: now also BUFFER-0A.A1; no longer IC1A.A1
- net PAGE-EN-A1: now also BUFFER-0A.A2; no longer IC1A.A2
- net PAGE-EN-A2: now also BUFFER-0A.A3; no longer IC1A.A3
- net PAGE-EN-A3: now also BUFFER-0A.A4; no longer IC1A.A4
- net PAGE-EN-B0: now also BUFFER-0A.B1; no longer IC1A.B1
- net PAGE-EN-B1: now also BUFFER-0A.B2; no longer IC1A.B2
- net PAGE-EN-B2: now also BUFFER-0A.B3; no longer IC1A.B3
- net PAGE-EN-B3: now also BUFFER-0A.B4; no longer IC1A.B4
- net VCC: now also BUFFER-0A.DIR, BUFFER-1A.DIR, BUFFER-3A.DIR; no longer IC1A.DIR, IC2A.DIR
- net WR: now also BUFFER-2A.DIR; no longer IC3A.DIR
Other:
- moved on the sheet: DEMUX-2X4-0A, MEMORY-0-8KX8-6264, MEMORY-1-8KX8-6264, MEMORY-2-8KX8-6264, MEMORY-3-8KX8-6264, PAGE-ADDR-REG-0

Commit message: Fixed address switch between prog and run modes for SRAM
Connections:
- net ADDR-C0 renamed ADDR-B0
- net ADDR-C1 renamed ADDR-B1
- net ADDR-C2 renamed ADDR-B2
- net ADDR-C3 renamed ADDR-B3
- net ADDR-C4 renamed ADDR-B4
- net ADDR-C5 renamed ADDR-B5
- net ADDR-C6 renamed ADDR-B6
- net ADDR-C7 renamed ADDR-B7
- net ADDR-C8 renamed ADDR-B8
- net ADDR-C9 renamed ADDR-B9
- removed net ADDR-D10: BUFFER-1A.B7, MEMORY-0-8KX8-6264.A10, MEMORY-1-8KX8-6264.A10, MEMORY-2-8KX8-6264.A10, MEMORY-3-8KX8-6264.A10
- removed net ADDR-D11: BUFFER-1A.B8, MEMORY-0-8KX8-6264.A11, MEMORY-1-8KX8-6264.A11, MEMORY-2-8KX8-6264.A11, MEMORY-3-8KX8-6264.A11
- removed net ADDR-D12: BUFFER-3A.B1, MEMORY-0-8KX8-6264.A12, MEMORY-1-8KX8-6264.A12, MEMORY-2-8KX8-6264.A12, MEMORY-3-8KX8-6264.A12
- new net ADDR-A10: ADDR-R/P-SW-2A.3Y, BUFFER-1A.A7, DEMUX-2X4-0A.A, LED15.A
- new net ADDR-A11: ADDR-R/P-SW-2A.4Y, BUFFER-1A.A8, DEMUX-2X4-0A.B, LED17.A
- new net ADDR-A12: ADDR-R/P-SW-3A.1Y, BUFFER-3A.A1, LED16.A
- net ADDR-B10: now also BUFFER-1A.B7, MEMORY-0-8KX8-6264.A10, MEMORY-1-8KX8-6264.A10, MEMORY-2-8KX8-6264.A10, MEMORY-3-8KX8-6264.A10; no longer ADDR-R/P-SW-2A.3Y, BUFFER-1A.A7, DEMUX-2X4-0A.A, LED15.A, PAGE-ADDR-REG-0A.Q1
- net ADDR-B11: now also BUFFER-1A.B8, MEMORY-0-8KX8-6264.A11, MEMORY-1-8KX8-6264.A11, MEMORY-2-8KX8-6264.A11, MEMORY-3-8KX8-6264.A11; no longer ADDR-R/P-SW-2A.4Y, BUFFER-1A.A8, DEMUX-2X4-0A.B, LED17.A, PAGE-ADDR-REG-0A.Q2
- net ADDR-B12: now also BUFFER-3A.B1, MEMORY-0-8KX8-6264.A12, MEMORY-1-8KX8-6264.A12, MEMORY-2-8KX8-6264.A12, MEMORY-3-8KX8-6264.A12; no longer ADDR-R/P-SW-3A.1Y, BUFFER-3A.A1, LED16.A, PAGE-ADDR-REG-0A.Q3
- net ADDR-R10: now also PAGE-ADDR-REG-0A.Q2
- net ADDR-R11: now also PAGE-ADDR-REG-0A.Q3
- net ADDR-R12: now also PAGE-ADDR-REG-0A.Q4
- net ADDR-R9: now also PAGE-ADDR-REG-0A.Q1
- net DATA-A0: now also PAGE-ADDR-REG-0A.D1
- net DATA-A1: now also PAGE-ADDR-REG-0A.D2
- net DATA-A2: now also PAGE-ADDR-REG-0A.D3
- net DATA-A3: now also PAGE-ADDR-REG-0A.D4
- net DATA-B0: no longer PAGE-ADDR-REG-0A.D1
- net DATA-B1: no longer PAGE-ADDR-REG-0A.D2
- net DATA-B2: no longer PAGE-ADDR-REG-0A.D3
- net DATA-B3: no longer PAGE-ADDR-REG-0A.D4
- net GND: no longer PAGE-ADDR-REG-0A.Q4
Other:
- moved on the sheet: ADDR-R/P-SW-0, ADDR-R/P-SW-1, ADDR-R/P-SW-2, ADDR-R/P-SW-3, BUFFER-0, BUFFER-1, BUFFER-2, BUFFER-3, DATA-R/P-SW-0, DATA-R/P-SW-1, DEMUX-2X4-0A, MEMORY-0-8KX8-6264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

Commit message: Fixed and improved schema for SRAM module
Connections:
- net ADDR-P0 renamed ADDR-PROG0
- net ADDR-P1 renamed ADDR-PROG1
- net ADDR-P10 renamed ADDR-PROG10
- net ADDR-P11 renamed ADDR-PROG11
- net ADDR-P12 renamed ADDR-PROG12
- net ADDR-P2 renamed ADDR-PROG2
- net ADDR-P3 renamed ADDR-PROG3
- net ADDR-P4 renamed ADDR-PROG4
- net ADDR-P5 renamed ADDR-PROG5
- net ADDR-P6 renamed ADDR-PROG6
- net ADDR-P7 renamed ADDR-PROG7
- net ADDR-P8 renamed ADDR-PROG8
- net ADDR-P9 renamed ADDR-PROG9
- net ADDR-R0 renamed ADDR-BUS0
- net ADDR-R1 renamed ADDR-BUS1
- net ADDR-R10 renamed ADDR-PAGE10
- net ADDR-R11 renamed ADDR-PAGE11
- net ADDR-R12 renamed ADDR-PAGE12
- net ADDR-R2 renamed ADDR-BUS2
- net ADDR-R3 renamed ADDR-BUS3
- net ADDR-R4 renamed ADDR-BUS4
- net ADDR-R5 renamed ADDR-BUS5
- net ADDR-R6 renamed ADDR-BUS6
- net ADDR-R7 renamed ADDR-BUS7
- net ADDR-R8 renamed ADDR-BUS8
- net ADDR-R9 renamed ADDR-PAGE9
- net DATA-P0 renamed DATA-PROG0
- net DATA-P1 renamed DATA-PROG1
- net DATA-P2 renamed DATA-PROG2
- net DATA-P3 renamed DATA-PROG3
- net DATA-P4 renamed DATA-PROG4
- net DATA-P5 renamed DATA-PROG5
- net DATA-P6 renamed DATA-PROG6
- net DATA-P7 renamed DATA-PROG7
- net DATA-R0 renamed DATA-BUS0
- net DATA-R1 renamed DATA-BUS1
- net DATA-R2 renamed DATA-BUS2
- net DATA-R3 renamed DATA-BUS3
- net DATA-R4 renamed DATA-BUS4
- net DATA-R5 renamed DATA-BUS5
- net DATA-R6 renamed DATA-BUS6
- net DATA-R7 renamed DATA-BUS7
- net PROG/RUN-SW renamed PROG/BUS-SW
- new net ADDR-BUS10: DEMUX-2X4-0A.B
- new net ADDR-BUS9: DEMUX-2X4-0A.A
- net ADDR-A10: no longer DEMUX-2X4-0A.A
- net ADDR-A11: no longer DEMUX-2X4-0A.B
Other:
- moved on the sheet: ADDR-R/P-SW-0, ADDR-R/P-SW-1, ADDR-R/P-SW-2, ADDR-R/P-SW-3, BUFFER-2, DATA-R/P-SW-0, DATA-R/P-SW-1, DEMUX-2X4-0A, MEMORY-0-8KX8-6264, MEMORY-1-8KX8-6264, MEMORY-2-8KX8-6264, MEMORY-3-8KX8-6264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

Commit message: Updated SRAM modules, unsed pins connected to the ground
Connections:
- net GND: now also ADDR-R/P-SW-3A.2A, ADDR-R/P-SW-3A.2B, ADDR-R/P-SW-3A.2Y, ADDR-R/P-SW-3A.3A, ADDR-R/P-SW-3A.3B, ADDR-R/P-SW-3A.3Y, ADDR-R/P-SW-3A.4A, ADDR-R/P-SW-3A.4B, ADDR-R/P-SW-3A.4Y, BUFFER-3A.A2, BUFFER-3A.A3, BUFFER-3A.A4, BUFFER-3A.A5, BUFFER-3A.A6, BUFFER-3A.A7, BUFFER-3A.A8, BUFFER-3A.B2, BUFFER-3A.B3, BUFFER-3A.B4, BUFFER-3A.B5, BUFFER-3A.B6, BUFFER-3A.B7, BUFFER-3A.B8
