File: ram/schema/rel-ram-4x8K.sch (EAGLE design)
At the start: 9 parts

Commit message: Added debug schema for SRAM circuit
Parts:
- removed PAGE-ADD-REG-1, PAGE-ADDR-REG-2, PAGE-ADDR-REG-3: 74LS173N, 74xx-eu:74LS173N
Connections:
- new net PR-LOAD: PAGE-ADDR-REG-0A.G1, PAGE-ADDR-REG-0A.G2
- net ADDR-B10: no longer PAGE-ADD-REG-1A.Q1, PAGE-ADDR-REG-2A.Q1, PAGE-ADDR-REG-3A.Q1
- net ADDR-B11: no longer PAGE-ADD-REG-1A.Q2, PAGE-ADDR-REG-2A.Q2, PAGE-ADDR-REG-3A.Q2
- net ADDR-B12: no longer PAGE-ADD-REG-1A.Q3, PAGE-ADDR-REG-2A.Q3, PAGE-ADDR-REG-3A.Q3
- net CLK-SIG: no longer PAGE-ADD-REG-1A.CLK, PAGE-ADDR-REG-2A.CLK, PAGE-ADDR-REG-3A.CLK
- net DATA0: no longer PAGE-ADD-REG-1A.D1, PAGE-ADDR-REG-2A.D1, PAGE-ADDR-REG-3A.D1
- net DATA1: no longer PAGE-ADD-REG-1A.D2, PAGE-ADDR-REG-2A.D2, PAGE-ADDR-REG-3A.D2
- net DATA2: no longer PAGE-ADD-REG-1A.D3, PAGE-ADDR-REG-2A.D3, PAGE-ADDR-REG-3A.D3
- net DATA3: now also PAGE-ADDR-REG-0A.D4; no longer PAGE-ADD-REG-1A.D4, PAGE-ADDR-REG-2A.D4, PAGE-ADDR-REG-3A.D4
- net DATA4: no longer PAGE-ADDR-REG-0A.D4
- net GND: no longer MEMORY-0-8KX8-6264.NC, MEMORY-1-8KX8-6264.NC, MEMORY-2-8KX8-6264.NC, MEMORY-3-8KX8-6264.NC, PAGE-ADD-REG-1A.CLR, PAGE-ADD-REG-1A.M, PAGE-ADD-REG-1A.N, PAGE-ADD-REG-1A.Q4, PAGE-ADDR-REG-2A.CLR, PAGE-ADDR-REG-2A.M, PAGE-ADDR-REG-2A.N, PAGE-ADDR-REG-2A.Q4, PAGE-ADDR-REG-3A.CLR, PAGE-ADDR-REG-3A.M, PAGE-ADDR-REG-3A.N, PAGE-ADDR-REG-3A.Q4
- net PAGE-EN0: no longer PAGE-ADDR-REG-0A.G1, PAGE-ADDR-REG-0A.G2
- net PAGE-EN1: no longer PAGE-ADD-REG-1A.G1, PAGE-ADD-REG-1A.G2
- net PAGE-EN2: no longer PAGE-ADDR-REG-2A.G1, PAGE-ADDR-REG-2A.G2
- net PAGE-EN3: no longer PAGE-ADDR-REG-3A.G1, PAGE-ADDR-REG-3A.G2
Other:
- moved on the sheet: DEMUX-2X4-0A, MEMORY-0-8KX8-6264, MEMORY-1-8KX8-6264, MEMORY-2-8KX8-6264, MEMORY-3-8KX8-6264, PAGE-ADDR-REG-0
