File: design/regs/schema/rel-regs.sch (EAGLE design)
At the start: 88 parts

Commit message: Aligned titles size for all schemas
Other:
- note added: "General Purpose Registers"
Changed lines of the file:
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@@
 <sheet>
 <plain>
+<wire x1="-182.88" y1="1371.6" x2="-182.88" y2="706.12" width="0.1524" layer="97" style="shortdash"/>
+<wire x1="-182.88" y1="706.12" x2="53.34" y2="706.12" width="0.1524" layer="97" style="shortdash"/>
+<wire x1="53.34" y1="706.12" x2="53.34" y2="1374.14" width="0.1524" layer="97" style="shortdash"/>
+<wire x1="53.34" y1="1374.14" x2="-182.88" y2="1374.14" width="0.1524" layer="97" style="shortdash"/>
+<wire x1="-182.88" y1="1374.14" x2="-182.88" y2="1371.6" width="0.1524" layer="97" style="shortdash"/>
+<text x="2.54" y="1369.06" size="2.54" layer="97">General Purpose Registers</text>
 </plain>
 <instances>

Commit message: Added initial description of General Purpose Registers to the HAS doc
Parts:
- renumbered REG-AC-BUF to REG-ACU-BUF, REG-AC-H to REG-ACU-H, REG-AC-L to REG-ACU-L
Connections:
- net REG-AC-DATA0 renamed REG-ACU-DATA0
- net REG-AC-DATA1 renamed REG-ACU-DATA1
- net REG-AC-DATA2 renamed REG-ACU-DATA2
- net REG-AC-DATA3 renamed REG-ACU-DATA3
- net REG-AC-DATA4 renamed REG-ACU-DATA4
- net REG-AC-DATA5 renamed REG-ACU-DATA5
- net REG-AC-DATA6 renamed REG-ACU-DATA6
- net REG-AC-DATA7 renamed REG-ACU-DATA7
