File: design/cu/schema/rel-cu.sch (EAGLE design)
At the start: 6 parts, among them IC2 74LS04N, IC3 74LS138N

Commit message: Fixed ustep connections for CU, added cmd codes and CPU flags
Parts:
- removed IC3: 74LS138N, 74xx-eu:74LS138N
- added AT28C16-3: (no value), memory:2816
- added IC1: 74154N, 74xx-eu:74154N
- added LED1, LED10, LED2, LED3, LED4, LED5, LED6, LED7, LED8, LED9: (no value), led:LED5MM
Connections:
- net IO3-I\ renamed ACU-O
- removed net USTEP0: AT28C16-0A.A0, AT28C16-1A.A0, AT28C16-2A.A0, IC3A.Y0
- removed net USTEP1: AT28C16-0A.A1, AT28C16-1A.A1, AT28C16-2A.A1, IC3A.Y1
- removed net USTEP2: AT28C16-0A.A2, AT28C16-1A.A2, AT28C16-2A.A2, IC3A.Y2
- removed net USTEP3: AT28C16-0A.A3, AT28C16-1A.A3, AT28C16-2A.A3, IC3A.Y3
- removed net USTEP4: AT28C16-0A.A4, AT28C16-1A.A4, AT28C16-2A.A4, IC3A.Y4
- removed net USTEP5: AT28C16-0A.A5, AT28C16-1A.A5, AT28C16-2A.A5, IC3A.Y5
- removed net USTEP6: AT28C16-0A.A6, AT28C16-1A.A6, AT28C16-2A.A6, IC3A.Y6
- removed net USTEP7: AT28C16-0A.A7, AT28C16-1A.A7, AT28C16-2A.A7, IC3A.Y7
- new net CF: AT28C16-0A.A4, AT28C16-1A.A4, AT28C16-2A.A4, AT28C16-3A.A4
- new net CMD0: AT28C16-0A.A7, AT28C16-1A.A7, AT28C16-2A.A7, AT28C16-3A.A7
- new net CMD1: AT28C16-0A.A8, AT28C16-1A.A8, AT28C16-2A.A8, AT28C16-3A.A8
- new net CMD2: AT28C16-0A.A9, AT28C16-1A.A9, AT28C16-2A.A9, AT28C16-3A.A9
- new net CMD3: AT28C16-0A.A10, AT28C16-1A.A10, AT28C16-2A.A10, AT28C16-3A.A10
- new net CS-I: AT28C16-3A.D4
- new net CU-RST: 74LS161NA.CLR, IC1A.10
- new net FLAG-I: AT28C16-3A.D5
- new net IO0-O: AT28C16-3A.D0
- new net IO1-O: AT28C16-3A.D1
- new net IO2-O: AT28C16-3A.D2
- new net IR-O: AT28C16-2A.D6
- new net MAR-O: AT28C16-2A.D5
- new net MBR-O: AT28C16-2A.D7
- new net N$10: IC1A.9, LED10.A
- new net N$4: IC1A.3, LED4.A
- new net N$5: IC1A.4, LED5.A
- new net N$6: IC1A.5, LED6.A
- new net N$7: IC1A.6, LED7.A
- new net N$8: IC1A.7, LED8.A
- new net N$9: IC1A.8, LED9.A
- new net PCL-I: AT28C16-3A.D3
- new net SF: AT28C16-0A.A5, AT28C16-1A.A5, AT28C16-2A.A5, AT28C16-3A.A5
- new net USTEP-A: 74LS161NA.QA, AT28C16-0A.A0, AT28C16-1A.A0, AT28C16-2A.A0, AT28C16-3A.A0, IC1A.A
- new net USTEP-B: 74LS161NA.QB, AT28C16-0A.A1, AT28C16-1A.A1, AT28C16-2A.A1, AT28C16-3A.A1, IC1A.B
- new net USTEP-C: 74LS161NA.QC, AT28C16-0A.A2, AT28C16-1A.A2, AT28C16-2A.A2, AT28C16-3A.A2, IC1A.C
- new net USTEP-D: 74LS161NA.QD, AT28C16-0A.A3, AT28C16-1A.A3, AT28C16-2A.A3, AT28C16-3A.A3, IC1A.D
- new net ZF: AT28C16-0A.A6, AT28C16-1A.A6, AT28C16-2A.A6, AT28C16-3A.A6
- net GND: now also AT28C16-3A.D6, AT28C16-3A.D7, IC1A.11, IC1A.12, IC1A.13, IC1A.14, IC1A.15, IC1A.G1, IC1A.G2, LED1.C, LED10.C, LED2.C, LED3.C, LED4.C, LED5.C, LED6.C, LED7.C, LED8.C, LED9.C; no longer 74LS161NA.QD, AT28C16-0A.A10, AT28C16-0A.A8, AT28C16-0A.A9, AT28C16-1A.A10, AT28C16-1A.A8, AT28C16-1A.A9, AT28C16-2A.A10, AT28C16-2A.A8, AT28C16-2A.A9, AT28C16-2A.D5, AT28C16-2A.D6, AT28C16-2A.D7, IC3A.G2A, IC3A.G2B
- net N$1: now also IC1A.0, LED1.A; no longer 74LS161NA.QA, IC3A.A
- net N$2: now also IC1A.1, LED2.A; no longer 74LS161NA.QB, IC3A.B
- net N$3: now also IC1A.2, LED3.A; no longer 74LS161NA.QC, IC3A.C
- net VCC: now also AT28C16-3A.!WE; no longer 74LS161NA.CLR, IC3A.G1
Other:
- moved on the sheet: 74LS161N, AT28C16-0, AT28C16-1, AT28C16-2

Commit message: Fixed CE OE signals for CU
Connections:
- net GND: now also AT28C16-3A.!CE, AT28C16-3A.!OE
Other:
- note added: "VER 1.1"
Changed lines of the file:
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@@
 <part name="AT28C16-3" library="memory" library_urn="urn:adsk.eagle:library:279" deviceset="2816" device="" package3d_urn="urn:adsk.eagle:package:19955/2"/>
 <part name="SUPPLY2" library="supply2" library_urn="urn:adsk.eagle:library:372" deviceset="VCC" device=""/>
+<part name="GND2" library="supply1" library_urn="urn:adsk.eagle:library:371" deviceset="GND" device=""/>
 </parts>
 <sheets>
@@
 <wire x1="-185.42" y1="449.58" x2="-185.42" y2="640.08" width="0.1524" layer="97" style="shortdash"/>
 <wire x1="-185.42" y1="640.08" x2="-434.34" y2="640.08" width="0.1524" layer="97" style="shortdash"/>
-<text x="-205.74" y="635" size="1.778" layer="97">CONTROL UNIT</text>
+<text x="-218.44" y="635" size="2.54" layer="97">CONTROL UNIT</text>
+<wire x1="-429.26" y1="469.9" x2="-429.26" y2="454.66" width="0.1524" layer="97"/>
+<wire x1="-429.26" y1="454.66" x2="-358.14" y2="454.66" width="0.1524" layer="97"/>
+<wire x1="-358.14" y1="454.66" x2="-358.14" y2="469.9" width="0.1524" layer="97"/>
+<wire x1="-358.14" y1="469.9" x2="-429.26" y2="469.9" width="0.1524" layer="97"/>
+<text x="-424.18" y="459.74" size="5.08" layer="97">VER 1.1</text>
 </plain>
 <instances>
@@
 <instance part="SUPPLY2" gate="G$1" x="-208.28" y="467.36" smashed="yes">
 <attribute name="VALUE" x="-210.185" y="470.535" size="1.778" layer="96"/>
+</instance>
+<instance part="GND2" gate="1" x="-243.84" y="462.28" smashed="yes">
+<attribute name="VALUE" x="-246.38" y="459.74" size="1.778" layer="96"/>
 </instance>
 </instances>
@@
 <junction x="-327.66" y="571.5"/>
 </segment>
+<segment>
+<pinref part="AT28C16-3" gate="A" pin="!OE"/>
+<wire x1="-236.22" y1="467.36" x2="-243.84" y2="467.36" width="0.1524" layer="91"/>
+<pinref part="AT28C16-3" gate="A" pin="!CE"/>
+<wire x1="-243.84" y1="467.36" x2="-243.84" y2="469.9" width="0.1524" layer="91"/>
+<wire x1="-243.84" y1="469.9" x2="-236.22" y2="469.9" width="0.1524" layer="91"/>
+<wire x1="-243.84" y1="467.36" x2="-243.84" y2="464.82" width="0.1524" layer="91"/>
+<junction x="-243.84" y="467.36"/>
+<pinref part="GND2" gate="1" pin="GND"/>
+</segment>
 </net>
